File: in_progress/pongclock/kicad/aw_601_pongclock.sch (KiCad schematic (older format))
At the start: 94 parts, among them CON1 BARREL_JACK, IC1 ATMEGA8-P, Q1 2N3904G, Q10 2N3904G, Q11 2N3904G, Q12 2N3904G, Q13 2N3904G, Q14 2N3904G, Q15 2N3904G, Q16 2N3904G, Q17 2N3904G, Q18 2N3904G, Q19 2N3904G, Q2 2N3904G, Q20 2N3904G, Q21 2N3904G, Q22 2N3904G, Q23 2N3904G, Q24 2N3904G, Q25 2N3904G, Q26 2N3904G, Q27 2N3904G, Q28 2N3904G, Q29 2N3904G, Q3 2N3904G, Q30 2N3904G, Q31 2N3904G, Q32 2N3904G, Q4 2N3904G, Q5 2N3904G, Q6 2N3904G, Q7 2N3904G, Q8 2N3904G, Q9 2N3904G, SW1 SW_PUSH, SW2 SW_PUSH, SW3 SW_PUSH, SW4 SW_PUSH, U1 4514, U10 DS1307, U2 ULN2803, U3 ULN2803, U4 ULN2803, U5 ULN2803, U6 74HC4094, U7 74HC4094, U8 74HC4094, U9 74HC4094, X1 16Mhz, X2 32kHz

Commit message: .
Parts:
- C1, C2: symbol C -> C-RESCUE-aw_601_pongclock
- C3: symbol CP1 -> CP1-RESCUE-aw_601_pongclock
- Q1, Q10, Q11, Q12, Q13, Q14, Q15, Q16, Q17, Q18, Q19, Q2, Q20, Q21, Q22, Q23, Q24, Q25, Q26, Q27, Q28, Q29, Q3, Q30, Q31, Q32, Q4, Q5, Q6, Q7, Q8, Q9: symbol PN2222A -> PN2222A-RESCUE-aw_601_pongclock
- R1, R10, R11, R12, R13, R2, R27, R28, R29, R3, R30, R31, R32, R33, R34, R35, R4, R5, R52, R53, R54, R55, R56, R57, R58, R59, R6, R60, R61, R62, R63, R64, R65, R66, R67, R7, R8, R9: symbol R -> R-RESCUE-aw_601_pongclock
