File: new/trainer/inputs.sch (KiCad schematic (older format))
At the start: 70 parts

Commit message: .
Parts:
- removed P?: CONN_2X2, SWITCHES, symbol CONN_2X2
- removed R? (x4): R, symbol R
- removed SW? (x4): SPST, ~, symbol SPST
- P?: footprint (none) -> Unbuffered switches
- P?: footprint (none) -> Buffered switches
Other:
- moved on the sheet: C?, P?, R?, RV?, SW?, U?A, U?B, U?C, U?D

Commit message: .
Parts:
- RV?: footprint ~ -> 5k
- RV? (x2): footprint ~ -> 10k
- RV?: footprint ~ -> 100k
Changed lines of the file:
@@
 LIBS:MiscellaneousDevices
 LIBS:ULN280xA
+LIBS:Gajda_cmosieee
+LIBS:jhd-162a
+LIBS:capteurs
 LIBS:trainer-cache
 EELAYER 25 0
@@
 F 0 "RV?" H 8700 2050 50  0000 C CNN
 F 1 "POT" H 8700 2150 50  0000 C CNN
-F 2 "~" H 8700 2150 60  0000 C CNN
+F 2 "5k" H 8600 2250 60  0000 C CNN
 F 3 "~" H 8700 2150 60  0000 C CNN
 	1    8700 2150
@@
 F 0 "RV?" H 9050 2050 50  0000 C CNN
 F 1 "POT" H 9050 2150 50  0000 C CNN
-F 2 "~" H 9050 2150 60  0000 C CNN
+F 2 "10k" H 8950 2250 60  0000 C CNN
 F 3 "~" H 9050 2150 60  0000 C CNN
 	1    9050 2150
@@
 F 0 "RV?" H 9400 2050 50  0000 C CNN
 F 1 "POT" H 9400 2150 50  0000 C CNN
-F 2 "~" H 9400 2150 60  0000 C CNN
+F 2 "10k" H 9300 2250 60  0000 C CNN
 F 3 "~" H 9400 2150 60  0000 C CNN
 	1    9400 2150
@@
 F 0 "RV?" H 9750 2050 50  0000 C CNN
 F 1 "POT" H 9750 2150 50  0000 C CNN
-F 2 "~" H 9750 2150 60  0000 C CNN
+F 2 "100k" H 9600 2250 60  0000 C CNN
 F 3 "~" H 9750 2150 60  0000 C CNN
 	1    9750 2150

Commit message: .
Parts:
- removed R? (x16): R, 10k, symbol R
Connections:
- net GNDREF: now also SW?.1, SW?.1, SW?.1, SW?.1, SW?.1, SW?.1, SW?.1, SW?.1, SW?.1, SW?.1, SW?.1, SW?.1, SW?.1, SW?.1, SW?.1, SW?.1
