File: new/trainer/outputs.sch (KiCad schematic (older format))
At the start: 0 parts

Commit message: .
Parts:
- added D? (x16): LED, symbol LED
- added P?: CONN_02X08, symbol CONN_02X08
- added R? (x16): R, 330R, symbol R
- added U? (x2): ULN2803A, symbol ULN2803A
Connections:
- net labels added: +5V, GNDREF
- wire segments 0 -> 77

Commit message: .
Parts:
- added AFF?: CA56-12, symbol CA56-12
- added IC?: ATTINY2313-P, DIP20, symbol ATTINY2313-P
- added P?: CONN_02X08, symbol CONN_02X08
- added P?: CONN_01X11, symbol CONN_01X11
- added Q? (x4): PN2222A, TO-92, symbol PN2222A
- added R? (x8): R, 390R, symbol R
- added RV?: POT, 10K, symbol POT
- added U?: 4067, symbol 4067
- added U?: JHD-162A, symbol JHD-162A
Connections:
- wire segments 77 -> 171
- no-connect marks 0 -> 2
Other:
- moved on the sheet: D?, P?, R?, U?

Commit message: .
Parts:
- removed Q? (x4): PN2222A, TO-92, symbol PN2222A
- added U?: ULN2803A, symbol ULN2803A
Connections:
- wire segments 171 -> 198
- no-connect marks 2 -> 4
Other:
- moved on the sheet: AFF?, D?, IC?, P?, R?, RV?, U?
