File: new/trainer/trainer.sch (KiCad schematic (older format))
At the start: 18 parts

Commit message: .
Parts:
- removed J?: USB, ~, symbol USB
- removed P?: CONN_4X2, POTS, symbol CONN_4X2
- removed P?: CONN_2X2, SWITCHES, symbol CONN_2X2
- removed P?: CONN_2X2, PUSHBUTTONS, symbol CONN_2X2
- removed RV? (x4): POT, ~, symbol POT
- removed SW? (x2): DUAL_SWITCH_INV, ~, symbol DUAL_SWITCH_INV
- removed SW? (x4): SPST, ~, symbol SPST
- removed SW?: SW_PUSH, ~, symbol SW_PUSH
- removed U?: 40106, symbol 40106
- added P?: USB_A, symbol USB_A
- added P?: CONN_01X04, symbol CONN_01X04
- added R? (x4): R, 10k, symbol R
- added S? (x4): RELAY_SPDT, symbol RELAY_SPDT
- added SW? (x2): Switch_SPDT_x2, symbol Switch_SPDT_x2
Connections:
- net labels added: GNDREF, R1_CLOSED, R1_COM, R1_OPEN, R2_CLOSED, R2_COM, R2_OPEN, R3_CLOSED, R3_COM, R3_OPEN, R4_CLOSED, R4_COM, R4_OPEN
- net labels removed: GND
- wire segments 47 -> 25
- no-connect marks 2 -> 1
Other:
- moved on the sheet: P?

Commit message: .
Parts:
- removed P?: CONN_2, POWER, symbol CONN_2
- removed P?: CONN_2, USB, symbol CONN_2
- removed R? (x4): R, 10k, symbol R
- removed SW? (x2): Switch_SPDT_x2, symbol Switch_SPDT_x2
- added C?: C, 0.33uF, symbol C
- added C?: C, 0.1uF, symbol C
- added CON?: BARREL_JACK, 7..12V, symbol BARREL_JACK
- added P?: CONN_01X03, USB, symbol CONN_01X03
- added P?: CONN_01X02, 5V to circuit, symbol CONN_01X02
- added P?: CONN_01X02, Power from circuit, symbol CONN_01X02
- added R? (x4): R, 220R, symbol R
- added U?: LM7805, symbol LM7805
- added U?: ULN2803A, symbol ULN2803A
- P?: footprint (none) -> RELAYS
Connections:
- net labels added: +5V
- wire segments 25 -> 44
Other:
- note added: "Isolated power supply\n(powers internal LEDs, ICs)"
- moved on the sheet: P?, S?

Commit message: .
Parts:
- added P?: CONN_01X03, symbol CONN_01X03
- added SP?: SPEAKER, symbol SPEAKER
- added X?: Buzzer_Son, symbol Buzzer_Son
Connections:
- wire segments 44 -> 51
Other:
- moved on the sheet: C?, CON?, P?, U?
Changed lines of the file:
@@
 LIBS:MiscellaneousDevices
 LIBS:ULN280xA
+LIBS:Gajda_cmosieee
+LIBS:jhd-162a
+LIBS:capteurs
 LIBS:trainer-cache
 EELAYER 25 0
@@
 L USB_A P?
 U 1 1 5653C819
-P 6650 1900
-F 0 "P?" H 6850 1700 50  0000 C CNN
-F 1 "USB_A" H 6600 2100 50  0000 C CNN
-F 2 "" V 6600 1800 60  0000 C CNN
-F 3 "" V 6600 1800 60  0000 C CNN
-	1    6650 1900
-	1    0    0    -1
-$EndComp
-NoConn ~ 6950 1800
+P 3600 900
+F 0 "P?" H 3800 700 50  0000 C CNN
+F 1 "USB_A" H 3550 1100 50  0000 C CNN
+F 2 "" V 3550 800 60  0000 C CNN
+F 3 "" V 3550 800 60  0000 C CNN
+	1    3600 900
+	1    0    0    -1
+$EndComp
+NoConn ~ 3900 800
 $Sheet
-S 8450 950  2150 1350
+S 5550 1300 2150 1350
 U 5655FD48
 F0 "Inputs" 60
@@
 $EndSheet
 $Sheet
-S 8450 2750 2150 1350
+S 8300 1300 2150 1350
 U 56560475
 F0 "Outputs" 60
@@
 L LM7805 U?
 U 1 1 5657C7C3
-P 2600 2350
-F 0 "U?" H 2750 2154 60  0000 C CNN
-F 1 "LM7805" H 2600 2550 60  0000 C CNN
-F 2 "" H 2600 2350 60  0000 C CNN
-F 3 "" H 2600 2350 60  0000 C CNN
-	1    2600 2350
+P 2500 2700
+F 0 "U?" H 2650 2504 60  0000 C CNN
+F 1 "LM7805" H 2500 2900 60  0000 C CNN
+F 2 "" H 2500 2700 60  0000 C CNN
+F 3 "" H 2500 2700 60  0000 C CNN
+	1    2500 2700
 	1    0    0    -1
 $EndComp
@@
 L GNDREF #PWR?
 U 1 1 5657D2EA
-P 6750 2750
-F 0 "#PWR?" H 6750 2500 50  0001 C CNN
-F 1 "GNDREF" H 6750 2600 50  0000 C CNN
-F 2 "" H 6750 2750 60  0000 C CNN
-F 3 "" H 6750 2750 60  0000 C CNN
-	1    6750 2750
+P 3700 1750
+F 0 "#PWR?" H 3700 1500 50  0001 C CNN
+F 1 "GNDREF" H 3700 1600 50  0000 C CNN
+F 2 "" H 3700 1750 60  0000 C CNN
+F 3 "" H 3700 1750 60  0000 C CNN
+	1    3700 1750
 	1    0    0    -1
 $EndComp
@@
 L C C?
 U 1 1 5657DDA5
-P 2200 2550
-F 0 "C?" H 2225 2650 50  0000 L CNN
-F 1 "C" H 2225 2450 50  0000 L CNN
-F 2 "0.33uF" H 2100 2450 30  0000 C CNN
-F 3 "" H 2200 2550 60  0000 C CNN
-	1    2200 2550
+P 2100 2900
+F 0 "C?" H 2125 3000 50  0000 L CNN
+F 1 "C" H 2125 2800 50  0000 L CNN
+F 2 "0.33uF" H 2000 2800 30  0000 C CNN
+F 3 "" H 2100 2900 60  0000 C CNN
+	1    2100 2900
 	1    0    0    -1
 $EndComp
@@
 L C C?
 U 1 1 5657DE9C
-P 3000 2550
-F 0 "C?" H 3025 2650 50  0000 L CNN
-F 1 "C" H 3025 2450 50  0000 L CNN
-F 2 "0.1uF" H 3150 2450 30  0000 C CNN
-F 3 "" H 3000 2550 60  0000 C CNN
-	1    3000 2550
+P 2900 2900
+F 0 "C?" H 2925 3000 50  0000 L CNN
+F 1 "C" H 2925 2800 50  0000 L CNN
+F 2 "0.1uF" H 3050 2800 30  0000 C CNN
+F 3 "" H 2900 2900 60  0000 C CNN
+	1    2900 2900
 	1    0    0    -1
 $EndComp
@@
 L GNDREF #PWR?
 U 1 1 5657E02B
-P 2600 2850
-F 0 "#PWR?" H 2600 2600 50  0001 C CNN
-F 1 "GNDREF" H 2600 2700 50  0000 C CNN
-F 2 "" H 2600 2850 60  0000 C CNN
-F 3 "" H 2600 2850 60  0000 C CNN
-	1    2600 2850
+P 2500 3200
+F 0 "#PWR?" H 2500 2950 50  0001 C CNN
+F 1 "GNDREF" H 2500 3050 50  0000 C CNN
+F 2 "" H 2500 3200 60  0000 C CNN
+F 3 "" H 2500 3200 60  0000 C CNN
+	1    2500 3200
 	1    0    0    -1
 $EndComp
@@
 L +5V #PWR?
 U 1 1 5657E06F
-P 3350 2150
-F 0 "#PWR?" H 3350 2000 50  0001 C CNN
-F 1 "+5V" H 3350 2290 50  0000 C CNN
-F 2 "" H 3350 2150 60  0000 C CNN
-F 3 "" H 3350 2150 60  0000 C CNN
-	1    3350 2150
+P 3250 2500
+F 0 "#PWR?" H 3250 2350 50  0001 C CNN
+F 1 "+5V" H 3250 2640 50  0000 C CNN
+F 2 "" H 3250 2500 60  0000 C CNN
+F 3 "" H 3250 2500 60  0000 C CNN
+	1    3250 2500
 	1    0    0    -1
 $EndComp
@@
 L BARREL_JACK CON?
 U 1 1 56587C69
-P 1450 2400
-F 0 "CON?" H 1450 2650 60  0000 C CNN
-F 1 "BARREL_JACK" H 1450 2200 60  0000 C CNN
-F 2 "7..12V" H 1450 2100 60  0000 C CNN
-F 3 "" H 1450 2400 60  0000 C CNN
-	1    1450 2400
+P 1350 2750
+F 0 "CON?" H 1350 3000 60  0000 C CNN
+F 1 "BARREL_JACK" H 1350 2550 60  0000 C CNN
+F 2 "7..12V" H 1350 2450 60  0000 C CNN
+F 3 "" H 1350 2750 60  0000 C CNN
+	1    1350 2750
 	1    0    0    -1
 $EndComp
@@
 L CONN_01X03 P?
 U 1 1 56588E62
-P 5950 2500
-F 0 "P?" H 5950 2700 50  0000 C CNN
-F 1 "CONN_01X03" V 6050 2500 50  0000 C CNN
-F 2 "USB" H 5950 2800 60  0000 C CNN
-F 3 "" H 5950 2500 60  0000 C CNN
-	1    5950 2500
+P 2900 1500
+F 0 "P?" H 2900 1700 50  0000 C CNN
+F 1 "CONN_01X03" V 3000 1500 50  0000 C CNN
+F 2 "USB" H 2900 1800 60  0000 C CNN
+F 3 "" H 2900 1500 60  0000 C CNN
+	1    2900 1500
 	-1   0    0    1
 $EndComp
@@
 L CONN_01X02 P?
 U 1 1 56589B7A
-P 3800 2350
-F 0 "P?" H 3800 2500 50  0000 C CNN
-F 1 "CONN_01X02" V 3900 2350 50  0000 C CNN
-F 2 "5V to circuit" H 3950 2050 60  0000 C CNN
-F 3 "" H 3800 2350 60  0000 C CNN
-	1    3800 2350
+P 3700 2700
+F 0 "P?" H 3700 2850 50  0000 C CNN
+F 1 "CONN_01X02" V 3800 2700 50  0000 C CNN
+F 2 "5V to circuit" H 3850 2400 60  0000 C CNN
+F 3 "" H 3700 2700 60  0000 C CNN
+	1    3700 2700
 	1    0    0    -1
 $EndComp
@@
 $EndComp
 Wire Wire Line
-	6550 2200 6550 2500
-Wire Wire Line
-	6650 2600 6650 2200
-Wire Wire Line
-	6750 2750 6750 2200
-Wire Wire Line
-	1750 2300 2200 2300
-Wire Wire Line
-	3000 2400 3000 2300
-Wire Wire Line
-	3000 2300 3600 2300
-Wire Wire Line
-	2200 2300 2200 2400
-Wire Wire Line
-	3350 2300 3350 2150
-Wire Wire Line
-	1750 2400 1750 2750
-Connection ~ 1750 2500
-Wire Wire Line
-	1750 2750 3600 2750
-Wire Wire Line
-	3000 2750 3000 2700
-Wire Wire Line
-	2600 2600 2600 2850
-Connection ~ 3000 2750
-Connection ~ 2600 2750
-Wire Wire Line
-	2200 2750 2200 2700
-Connection ~ 2200 2750
-Wire Wire Line
-	6550 2500 6150 2500
-Wire Wire Line
-	6150 2600 6650 2600
-Wire Wire Line
-	6150 2400 6450 2400
-Wire Wire Line
-	6450 2400 6450 2200
-Connection ~ 3350 2300
-Wire Wire Line
-	3600 2750 3600 2400
+	3500 1200 3500 1500
+Wire Wire Line
+	3600 1600 3600 1200
+Wire Wire Line
+	3700 1750 3700 1200
+Wire Wire Line
+	1650 2650 2100 2650
+Wire Wire Line
+	2900 2750 2900 2650
+Wire Wire Line
+	2900 2650 3500 2650
+Wire Wire Line
+	2100 2650 2100 2750
+Wire Wire Line
+	3250 2650 3250 2500
+Wire Wire Line
+	1650 2750 1650 3100
+Connection ~ 1650 2850
+Wire Wire Line
+	1650 3100 3500 3100
+Wire Wire Line
+	2900 3100 2900 3050
+Wire Wire Line
+	2500 2950 2500 3200
+Connection ~ 2900 3100
+Connection ~ 2500 3100
+Wire Wire Line
+	2100 3100 2100 3050
+Connection ~ 2100 3100
+Wire Wire Line
+	3500 1500 3100 1500
+Wire Wire Line
+	3100 1600 3600 1600
+Wire Wire Line
+	3100 1400 3400 1400
+Wire Wire Line
+	3400 1400 3400 1200
+Connection ~ 3250 2650
+Wire Wire Line
+	3500 3100 3500 2750
 Wire Wire Line
 	3000 4800 3100 4800
@@
 Wire Wire Line
 	1350 1300 1500 1300
-Text Notes 1900 3300 0    60   ~ 0
+Text Notes 1800 3650 0    60   ~ 0
 Isolated power supply\n(powers internal LEDs, ICs)
+$Comp
+L CONN_01X03 P?
+U 1 1 565A63D3
+P 8400 3900
+F 0 "P?" H 8400 4100 50  0000 C CNN
+F 1 "CONN_01X03" V 8500 3900 50  0000 C CNN
+F 2 "" H 8400 3900 60  0000 C CNN
+F 3 "" H 8400 3900 60  0000 C CNN
+	1    8400 3900
+	1    0    0    -1
+$EndComp
+$Comp
+L SPEAKER SP?
+U 1 1 565A67F9
+P 7450 3800
+F 0 "SP?" H 7350 4050 50  0000 C CNN
+F 1 "SPEAKER" H 7350 3550 50  0000 C CNN
+F 2 "" H 7450 3800 60  0000 C CNN
+F 3 "" H 7450 3800 60  0000 C CNN
+	1    7450 3800
+	-1   0    0    1
+$EndComp
+$Comp
+L Buzzer_Son X?
+U 1 1 565A69C0
+P 7550 4450
+F 0 "X?" H 7400 4700 60  0000 C CNN
+F 1 "Buzzer_Son" H 7800 4700 60  0000 C CNN
+F 2 "" H 7550 4450 60  0000 C CNN
+F 3 "" H 7550 4450 60  0000 C CNN
+	1    7550 4450
+	1    0    0    -1
+$EndComp
+Wire Wire Line
+	8200 3900 7750 3900
+Wire Wire Line
+	8200 4000 8200 4350
+Wire Wire Line
+	8200 4350 7850 4350
+Wire Wire Line
+	7750 3700 8200 3700
+Wire Wire Line
+	8200 3700 8200 3800
+Wire Wire Line
+	7850 4550 8200 4550
+Wire Wire Line
+	8200 4550 8200 4650
+$Comp
+L GNDREF #PWR?
+U 1 1 565A72DA
+P 8200 4650
+F 0 "#PWR?" H 8200 4400 50  0001 C CNN
+F 1 "GNDREF" H 8200 4500 50  0000 C CNN
+F 2 "" H 8200 4650 60  0000 C CNN
+F 3 "" H 8200 4650 60  0000 C CNN
+	1    8200 4650
+	1    0    0    -1
+$EndComp
 $EndSCHEMATC

Commit message: .
Parts:
- added Q?: PN2222A, TO-92, symbol PN2222A
- added R?: R, 1K, symbol R
Connections:
- wire segments 51 -> 61
Other:
- note added: "TODO - use the same ULN2803 \nused in the 7-digit seg display."
- moved on the sheet: P?, SP?, X?
Changed lines of the file:
@@
 LIBS:memory
 LIBS:xilinx
+LIBS:special
 LIBS:microcontrollers
 LIBS:dsp
@@
 LIBS:valves
 LIBS:MiscellaneousDevices
-LIBS:ULN280xA
 LIBS:Gajda_cmosieee
 LIBS:jhd-162a
 LIBS:capteurs
 LIBS:trainer-cache
-EELAYER 25 0
+EELAYER 27 0
 EELAYER END
 $Descr A4 11693 8268
@@
 Sheet 1 3
 Title ""
-Date "22 nov 2015"
+Date "29 nov 2015"
 Rev ""
 Comp ""
@@
 	2900 2750 2900 2650
 Wire Wire Line
-	2900 2650 3500 2650
+	2900 2650 3250 2650
+Wire Wire Line
+	3250 2650 3500 2650
 Wire Wire Line
 	2100 2650 2100 2750
@@
 	3250 2650 3250 2500
 Wire Wire Line
-	1650 2750 1650 3100
+	1650 2750 1650 2850
+Wire Wire Line
+	1650 2850 1650 3100
 Connection ~ 1650 2850
 Wire Wire Line
-	1650 3100 3500 3100
+	1650 3100 2100 3100
+Wire Wire Line
+	2100 3100 2500 3100
+Wire Wire Line
+	2500 3100 2900 3100
+Wire Wire Line
+	2900 3100 3500 3100
 Wire Wire Line
 	2900 3100 2900 3050
 Wire Wire Line
-	2500 2950 2500 3200
+	2500 2950 2500 3100
+Wire Wire Line
+	2500 3100 2500 3200
 Connection ~ 2900 3100
 Connection ~ 2500 3100
@@
 	3000 5100 3100 5100
 Wire Wire Line
-	4000 3950 4000 6600
+	4000 3950 4000 4200
+Wire Wire Line
+	4000 4200 4000 5000
+Wire Wire Line
+	4000 5000 4000 5800
+Wire Wire Line
+	4000 5800 4000 6600
 Wire Wire Line
 	4000 4200 4200 4200
@@
 L CONN_01X03 P?
 U 1 1 565A63D3
-P 8400 3900
-F 0 "P?" H 8400 4100 50  0000 C CNN
-F 1 "CONN_01X03" V 8500 3900 50  0000 C CNN
-F 2 "" H 8400 3900 60  0000 C CNN
-F 3 "" H 8400 3900 60  0000 C CNN
-	1    8400 3900
+P 10250 3700
+F 0 "P?" H 10250 3900 50  0000 C CNN
+F 1 "CONN_01X03" V 10350 3700 50  0000 C CNN
+F 2 "" H 10250 3700 60  0000 C CNN
+F 3 "" H 10250 3700 60  0000 C CNN
+	1    10250 3700
 	1    0    0    -1
 $EndComp
@@
 L SPEAKER SP?
 U 1 1 565A67F9
-P 7450 3800
-F 0 "SP?" H 7350 4050 50  0000 C CNN
-F 1 "SPEAKER" H 7350 3550 50  0000 C CNN
-F 2 "" H 7450 3800 60  0000 C CNN
-F 3 "" H 7450 3800 60  0000 C CNN
-	1    7450 3800
+P 9300 3600
+F 0 "SP?" H 9200 3850 50  0000 C CNN
+F 1 "SPEAKER" H 9200 3350 50  0000 C CNN
+F 2 "" H 9300 3600 60  0000 C CNN
+F 3 "" H 9300 3600 60  0000 C CNN
+	1    9300 3600
 	-1   0    0    1
 $EndComp
@@
 L Buzzer_Son X?
 U 1 1 565A69C0
-P 7550 4450
-F 0 "X?" H 7400 4700 60  0000 C CNN
-F 1 "Buzzer_Son" H 7800 4700 60  0000 C CNN
-F 2 "" H 7550 4450 60  0000 C CNN
-F 3 "" H 7550 4450 60  0000 C CNN
-	1    7550 4450
-	1    0    0    -1
-$EndComp
-Wire Wire Line
-	8200 3900 7750 3900
-Wire Wire Line
-	8200 4000 8200 4350
-Wire Wire Line
-	8200 4350 7850 4350
-Wire Wire Line
-	7750 3700 8200 3700
-Wire Wire Line
-	8200 3700 8200 3800
-Wire Wire Line
-	7850 4550 8200 4550
-Wire Wire Line
-	8200 4550 8200 4650
+P 8350 3950
+F 0 "X?" H 8200 4200 60  0000 C CNN
+F 1 "Buzzer_Son" H 8600 4200 60  0000 C CNN
+F 2 "" H 8350 3950 60  0000 C CNN
+F 3 "" H 8350 3950 60  0000 C CNN
+	1    8350 3950
+	1    0    0    -1
+$EndComp
+Wire Wire Line
+	10050 3700 9600 3700
+Wire Wire Line
+	9600 3500 10050 3500
+Wire Wire Line
+	10050 3500 10050 3600
+$Comp
+L +5V #PWR?
+U 1 1 565B1AC3
+P 8650 3450
+F 0 "#PWR?" H 8650 3300 50  0001 C CNN
+F 1 "+5V" H 8650 3590 50  0000 C CNN
+F 2 "" H 8650 3450 60  0000 C CNN
+F 3 "" H 8650 3450 60  0000 C CNN
+	1    8650 3450
+	1    0    0    -1
+$EndComp
+Wire Wire Line
+	8650 3450 8650 3850
+$Comp
+L PN2222A Q?
+U 1 1 565B1B0C
+P 8750 4250
+F 0 "Q?" H 8950 4325 50  0000 L CNN
+F 1 "PN2222A" H 8950 4250 50  0000 L CNN
+F 2 "TO-92" H 8950 4175 50  0000 L CIN
+F 3 "" H 8750 4250 50  0000 L CNN
+	1    8750 4250
+	-1   0    0    -1
+$EndComp
 $Comp
 L GNDREF #PWR?
-U 1 1 565A72DA
-P 8200 4650
-F 0 "#PWR?" H 8200 4400 50  0001 C CNN
-F 1 "GNDREF" H 8200 4500 50  0000 C CNN
-F 2 "" H 8200 4650 60  0000 C CNN
-F 3 "" H 8200 4650 60  0000 C CNN
-	1    8200 4650
-	1    0    0    -1
-$EndComp
+U 1 1 565B1B2B
+P 8650 4550
+F 0 "#PWR?" H 8650 4300 50  0001 C CNN
+F 1 "GNDREF" H 8650 4400 50  0000 C CNN
+F 2 "" H 8650 4550 60  0000 C CNN
+F 3 "" H 8650 4550 60  0000 C CNN
+	1    8650 4550
+	1    0    0    -1
+$EndComp
+Wire Wire Line
+	8650 4450 8650 4550
+$Comp
+L R R?
+U 1 1 565B1BAF
+P 9400 4250
+F 0 "R?" V 9480 4250 40  0000 C CNN
+F 1 "R" V 9407 4251 40  0000 C CNN
+F 2 "1K" V 9330 4250 30  0000 C CNN
+F 3 "~" H 9400 4250 30  0000 C CNN
+	1    9400 4250
+	0    -1   -1   0
+$EndComp
+Wire Wire Line
+	8950 4250 9150 4250
+Wire Wire Line
+	9650 4250 10050 4250
+Wire Wire Line
+	10050 4250 10050 3800
+Text Notes 8400 5000 0    60   ~ 0
+TODO - use the same ULN2803 \nused in the 7-digit seg display.
 $EndSCHEMATC
