File: done/power_supply/power_supply.sch (KiCad schematic (older format))
At the start: 4 parts

Commit message: .
Parts:
- added C1, C5, C6: CP1, 10uF 50V, symbol CP1
- added C2: CP1, 2200uF 50V, symbol CP1
- added C3: CP1, 100uF 25V, symbol CP1
- added C4: C, 100nF 50V, symbol C
- added D1: LED, ~, symbol LED
- added D10, D11, D12, D2, D3, D4, D5, D6, D7, D9: DIODE, 1N4007, symbol DIODE
- added D8: ZENER, 6V2, symbol ZENER
- added R1: R, 10K, symbol R
- added R2: R, 82R, symbol R
- added R3: R, 10K 1/2W, symbol R
- added R4: R, 220R, symbol R
- added R5, R7: R, 240R, symbol R
- added R6: R, 1R 5W, symbol R
- added RV1: POT, 1K linear, symbol POT
- added RV2: POT, 10K linear, symbol POT
- added U1, U3: LM317T, TO-220, symbol LM317T
- added U2: LM317L, TO-92, symbol LM317H
- added U4: YB27VA, symbol YB27VA
- gave numbers to parts that had none: 4
Connections:
- net labels added: +5V, Independent power, MAINS, S1, S2, V+
- net labels removed: +18VAC, 110/220VAC, NEUTRAL
- wire segments 11 -> 64
Other:
- moved on the sheet: F1, SW1, SW2A, T1

Commit message: .
Parts:
- C1, C2, C3, C5, C6: symbol CP1 -> CP1-RESCUE-power_supply
- C4: symbol C -> C-RESCUE-power_supply
- D1: symbol LED -> LED-RESCUE-power_supply
- D8: symbol ZENER -> ZENER-RESCUE-power_supply
- R1, R2, R3, R4, R5, R6, R7: symbol R -> R-RESCUE-power_supply
Connections:
- net GND: no longer D8.1 (A), R4.2, R5.1, U2.1 (IN)
- new net: D8.1 (A), R4.2, R5.1, U2.1 (IN)
Changed lines of the file:
@@
 EESchema Schematic File Version 2
+LIBS:power_supply-rescue
 LIBS:power
 LIBS:device
@@
 LIBS:valves
 LIBS:power_supply-cache
-EELAYER 27 0
+EELAYER 25 0
 EELAYER END
 $Descr A4 11693 8268
@@
 110VAC
 $Comp
-L R R1
+L R-RESCUE-power_supply R1
 U 1 1 56509E9F
 P 1750 4050
@@
 $EndComp
 $Comp
-L LED D1
+L LED-RESCUE-power_supply D1
 U 1 1 56509EAE
 P 1750 4750
@@
 $EndComp
 $Comp
-L R R2
+L R-RESCUE-power_supply R2
 U 1 1 56509FF0
 P 2000 5550
@@
 $EndComp
 $Comp
-L CP1 C1
+L CP1-RESCUE-power_supply C1
 U 1 1 5651B086
 P 2450 5550
@@
 $EndComp
 $Comp
-L R R3
+L R-RESCUE-power_supply R3
 U 1 1 5651B12C
 P 2950 4450
@@
 $EndComp
 $Comp
-L CP1 C2
+L CP1-RESCUE-power_supply C2
 U 1 1 5651B13B
 P 3300 4450
@@
 $EndComp
 $Comp
-L C C4
+L C-RESCUE-power_supply C4
 U 1 1 5651B154
 P 3800 4450
@@
 $EndComp
 $Comp
-L CP1 C3
+L CP1-RESCUE-power_supply C3
 U 1 1 5651B195
 P 3300 5350
@@
 $EndComp
 $Comp
-L R R4
+L R-RESCUE-power_supply R4
 U 1 1 5651B1AE
 P 3550 5550
@@
 $EndComp
 $Comp
-L ZENER D8
+L ZENER-RESCUE-power_supply D8
 U 1 1 5651B1C7
 P 3800 5350
@@
 $EndComp
 $Comp
-L R R6
+L R-RESCUE-power_supply R6
 U 1 1 5651B3DC
 P 4850 3800
@@
 $EndComp
 $Comp
-L R R5
+L R-RESCUE-power_supply R5
 U 1 1 5651B499
 P 4400 4900
@@
 $EndComp
 $Comp
-L R R7
+L R-RESCUE-power_supply R7
 U 1 1 5651BE45
 P 6850 4050
@@
 $EndComp
 $Comp
-L CP1 C5
+L CP1-RESCUE-power_supply C5
 U 1 1 5651C070
 P 6500 4750
@@
 $EndComp
 $Comp
-L CP1 C6
+L CP1-RESCUE-power_supply C6
 U 1 1 5651C238
 P 7300 4450
@@
 $EndComp
 $Comp
-L GND #PWR1
+L GND-RESCUE-power_supply #PWR1
 U 1 1 5651C384
 P 6050 5300
@@
 Wire Wire Line
 	2250 5150 9500 5150
-Connection ~ 4150 5150
 Wire Wire Line
 	4200 4200 4200 4100
@@
 $EndComp
 $Comp
-L GND #PWR3
+L GND-RESCUE-power_supply #PWR3
 U 1 1 5651D109
 P 8200 4850
