File: in_progress/led_dimmer/dimmer.sch (KiCad schematic (older format))
At the start: 19 parts, among them Q1 2N3904, SW1 SPST, U1 NE555

Commit message: .
Parts:
- U1: symbol LM555N -> LM555N-RESCUE-dimmer
Changed lines of the file:
@@
 EESchema Schematic File Version 2
+LIBS:dimmer-rescue
 LIBS:power
 LIBS:device
@@
 $EndComp
 $Comp
-L LM555N U1
+L LM555N-RESCUE-dimmer U1
 U 1 1 56741A2A
 P 5050 4000
