File: in_progress/led_dimmer/led_dimmer.sch (KiCad schematic (older format))
At the start: 21 parts, among them IC1 ATTINY2313A-P, Q1 Q_NPN_CBE, SW1 SPST

Commit message: .
Parts:
- removed R1: R, 45k, symbol R
- removed R10, R9: R, 10k, symbol R
- removed R11, R12, R13: R, 100R, symbol R
- removed R2: R, 15k, symbol R
- removed R3: R, 8k, symbol R
- removed R4: R, 4k5, symbol R
- removed R5: R, 3k, symbol R
- removed R6: R, 2k, symbol R
- removed R7: R, 1k7, symbol R
- removed R8: R, 1k2, symbol R
- added C? (x2): C, 22pF, symbol C
- added C?: CP1, 0.1uF, symbol CP1
- added C?: C, 0.1uF, symbol C
- added C?: CP1, 10uF, symbol CP1
- added P?: CONN_3X2, symbol CONN_3X2
- added P? (x2): CONN_4, symbol CONN_4
- added R?: R, 10k, symbol R-RESCUE-led_dimmer
- added R? (x2): R, 10k, symbol R
- added R? (x9): R, 68R, symbol R-RESCUE-led_dimmer
- added X?: CRYSTAL, 8 MHz, symbol CRYSTAL
- D1, D2, D3: symbol LED -> LED-RESCUE-led_dimmer
- RV1: footprint (none) -> 100k
Connections:
- wire segments 45 -> 70
- no-connect marks 6 -> 0
Other:
- moved on the sheet: BT1, IC1, Q1, RV1, SW1

Commit message: .
Parts:
- C1, C5: renamed from C?; symbol CP1 -> CP1-RESCUE-led_dimmer
- C2, C3, C4: renamed from C?; symbol C -> C-RESCUE-led_dimmer
- R2, R3: renamed from R?; symbol R -> R-RESCUE-led_dimmer
- gave numbers to parts that had none: 14
Changed lines of the file:
@@
 $EndComp
 $Comp
-L GND-RESCUE-led_dimmer #PWR02
+L GND-RESCUE-led_dimmer #PWR10
 U 1 1 56624E68
 P 5550 2450
-F 0 "#PWR02" H 5550 2200 50  0001 C CNN
+F 0 "#PWR10" H 5550 2200 50  0001 C CNN
 F 1 "GND" H 5550 2300 50  0000 C CNN
 F 2 "" H 5550 2450 50  0000 C CNN
@@
 $EndComp
 $Comp
-L VCC #PWR05
+L VCC #PWR6
 U 1 1 566286D5
 P 4350 1950
-F 0 "#PWR05" H 4350 1800 50  0001 C CNN
+F 0 "#PWR6" H 4350 1800 50  0001 C CNN
 F 1 "VCC" H 4350 2100 50  0000 C CNN
 F 2 "" H 4350 1950 50  0000 C CNN
@@
 $EndComp
 $Comp
-L GND-RESCUE-led_dimmer #PWR06
+L GND-RESCUE-led_dimmer #PWR7
 U 1 1 566287A3
 P 4350 4750
-F 0 "#PWR06" H 4350 4500 50  0001 C CNN
+F 0 "#PWR7" H 4350 4500 50  0001 C CNN
 F 1 "GND" H 4350 4600 50  0000 C CNN
 F 2 "" H 4350 4750 50  0000 C CNN
@@
 $EndComp
 $Comp
-L VCC #PWR07
+L VCC #PWR4
 U 1 1 56628A26
 P 2950 2650
-F 0 "#PWR07" H 2950 2500 50  0001 C CNN
+F 0 "#PWR4" H 2950 2500 50  0001 C CNN
 F 1 "VCC" H 2950 2800 50  0000 C CNN
 F 2 "" H 2950 2650 50  0000 C CNN
@@
 $EndComp
 $Comp
-L VCC #PWR08
+L VCC #PWR1
 U 1 1 56628B36
 P 1750 2800
-F 0 "#PWR08" H 1750 2650 50  0001 C CNN
+F 0 "#PWR1" H 1750 2650 50  0001 C CNN
 F 1 "VCC" H 1750 2950 50  0000 C CNN
 F 2 "" H 1750 2800 50  0000 C CNN
@@
 $EndComp
 $Comp
-L GND-RESCUE-led_dimmer #PWR09
+L GND-RESCUE-led_dimmer #PWR2
 U 1 1 56628B68
 P 1750 4300
-F 0 "#PWR09" H 1750 4050 50  0001 C CNN
+F 0 "#PWR2" H 1750 4050 50  0001 C CNN
 F 1 "GND" H 1750 4150 50  0000 C CNN
 F 2 "" H 1750 4300 50  0000 C CNN
@@
 $EndComp
 $Comp
-L VCC #PWR010
+L VCC #PWR14
 U 1 1 5662A328
 P 7750 1650
-F 0 "#PWR010" H 7750 1500 50  0001 C CNN
+F 0 "#PWR14" H 7750 1500 50  0001 C CNN
 F 1 "VCC" H 7750 1800 50  0000 C CNN
 F 2 "" H 7750 1650 50  0000 C CNN
@@
 $EndComp
 $Comp
-L GND-RESCUE-led_dimmer #PWR011
+L GND-RESCUE-led_dimmer #PWR15
 U 1 1 5662A7BE
 P 8450 4050
-F 0 "#PWR011" H 8450 3800 50  0001 C CNN
+F 0 "#PWR15" H 8450 3800 50  0001 C CNN
 F 1 "GND" H 8450 3900 50  0000 C CNN
 F 2 "" H 8450 4050 50  0000 C CNN
@@
 $EndComp
 $Comp
-L CRYSTAL X?
+L CRYSTAL X1
 U 1 1 567D3088
 P 2700 3450
-F 0 "X?" H 2700 3600 60  0000 C CNN
+F 0 "X1" H 2700 3600 60  0000 C CNN
 F 1 "CRYSTAL" H 2700 3300 60  0000 C CNN
 F 2 "8 MHz" H 2700 3700 60  0000 C CNN
@@
 $EndComp
 $Comp
-L C C?
+L C-RESCUE-led_dimmer C3
 U 1 1 567D3309
 P 2950 3650
-F 0 "C?" H 2950 3750 40  0000 L CNN
+F 0 "C3" H 2950 3750 40  0000 L CNN
 F 1 "C" H 2956 3565 40  0000 L CNN
 F 2 "22pF" H 3000 3500 30  0000 C CNN
@@
 $EndComp
 $Comp
-L C C?
+L C-RESCUE-led_dimmer C2
 U 1 1 567D336C
 P 2400 3650
-F 0 "C?" H 2400 3750 40  0000 L CNN
+F 0 "C2" H 2400 3750 40  0000 L CNN
 F 1 "C" H 2406 3565 40  0000 L CNN
 F 2 "22pF" H 2450 3500 30  0000 C CNN
@@
 $EndComp
 $Comp
-L GND #PWR?
+L GND-RESCUE-led_dimmer #PWR3
 U 1 1 567D33C8
 P 2400 3850
-F 0 "#PWR?" H 2400 3850 30  0001 C CNN
+F 0 "#PWR3" H 2400 3850 30  0001 C CNN
 F 1 "GND" H 2400 3780 30  0001 C CNN
 F 2 "" H 2400 3850 60  0000 C CNN
@@
 $EndComp
 $Comp
-L GND #PWR?
+L GND-RESCUE-led_dimmer #PWR5
 U 1 1 567D3407
 P 2950 3850
-F 0 "#PWR?" H 2950 3850 30  0001 C CNN
+F 0 "#PWR5" H 2950 3850 30  0001 C CNN
 F 1 "GND" H 2950 3780 30  0001 C CNN
 F 2 "" H 2950 3850 60  0000 C CNN
@@
 $EndComp
 $Comp
-L CP1 C?
+L CP1-RESCUE-led_dimmer C5
 U 1 1 567D430D
 P 6500 3500
-F 0 "C?" H 6550 3600 50  0000 L CNN
+F 0 "C5" H 6550 3600 50  0000 L CNN
 F 1 "CP1" H 6550 3400 50  0000 L CNN
 F 2 "0.1uF" H 6750 3500 60  0000 C CNN
@@
 $EndComp
 $Comp
-L GND #PWR?
+L GND-RESCUE-led_dimmer #PWR11
 U 1 1 567D4375
 P 6500 3700
-F 0 "#PWR?" H 6500 3700 30  0001 C CNN
+F 0 "#PWR11" H 6500 3700 30  0001 C CNN
 F 1 "GND" H 6500 3630 30  0001 C CNN
 F 2 "" H 6500 3700 60  0000 C CNN
@@
 $EndComp
 $Comp
-L VCC #PWR?
+L VCC #PWR9
 U 1 1 567D5148
 P 5550 1650
-F 0 "#PWR?" H 5550 1500 50  0001 C CNN
+F 0 "#PWR9" H 5550 1500 50  0001 C CNN
 F 1 "VCC" H 5550 1800 50  0000 C CNN
 F 2 "" H 5550 1650 50  0000 C CNN
@@
 $EndComp
 $Comp
-L R-RESCUE-led_dimmer R?
+L R-RESCUE-led_dimmer R1
 U 1 1 567D51AB
 P 5550 1800
-F 0 "R?" V 5650 1800 50  0000 C CNN
+F 0 "R1" V 5650 1800 50  0000 C CNN
 F 1 "R" V 5550 1800 50  0000 C CNN
 F 2 "10k" V 5450 1800 50  0000 C CNN
@@
 $EndComp
 $Comp
-L R R?
+L R-RESCUE-led_dimmer R3
 U 1 1 567D5281
 P 6900 2250
-F 0 "R?" V 6980 2250 40  0000 C CNN
+F 0 "R3" V 6980 2250 40  0000 C CNN
 F 1 "R" V 6907 2251 40  0000 C CNN
 F 2 "10k" V 6830 2250 30  0000 C CNN
@@
 $EndComp
 $Comp
-L R R?
+L R-RESCUE-led_dimmer R2
 U 1 1 567D54F3
 P 6100 3250
-F 0 "R?" V 6180 3250 40  0000 C CNN
+F 0 "R2" V 6180 3250 40  0000 C CNN
 F 1 "R" V 6107 3251 40  0000 C CNN
 F 2 "10k" V 6030 3250 30  0000 C CNN
@@
 $EndComp
 $Comp
-L CONN_3X2 P?
+L CONN_3X2 P1
 U 1 1 567D6308
 P 6800 4300
-F 0 "P?" H 6800 4550 50  0000 C CNN
+F 0 "P1" H 6800 4550 50  0000 C CNN
 F 1 "CONN_3X2" V 6800 4350 40  0000 C CNN
 F 2 "" H 6800 4300 60  0000 C CNN
@@
 $EndComp
 $Comp
-L VCC #PWR?
+L VCC #PWR12
 U 1 1 567D678E
 P 7200 3750
-F 0 "#PWR?" H 7200 3600 50  0001 C CNN
+F 0 "#PWR12" H 7200 3600 50  0001 C CNN
 F 1 "VCC" H 7200 3900 50  0000 C CNN
 F 2 "" H 7200 3750 50  0000 C CNN
@@
 $EndComp
 $Comp
-L GND #PWR?
+L GND-RESCUE-led_dimmer #PWR13
 U 1 1 567D67D2
 P 7200 4550
-F 0 "#PWR?" H 7200 4550 30  0001 C CNN
+F 0 "#PWR13" H 7200 4550 30  0001 C CNN
 F 1 "GND" H 7200 4480 30  0001 C CNN
 F 2 "" H 7200 4550 60  0000 C CNN
@@
 $EndComp
 $Comp
-L R-RESCUE-led_dimmer R?
+L R-RESCUE-led_dimmer R4
 U 1 1 567D6D84
 P 7650 2950
-F 0 "R?" V 7700 3150 50  0000 C CNN
+F 0 "R4" V 7700 3150 50  0000 C CNN
 F 1 "R" V 7650 2950 50  0000 C CNN
 F 2 "68R" V 7700 2700 50  0000 C CNN
@@
 $EndComp
 $Comp
-L R-RESCUE-led_dimmer R?
+L R-RESCUE-led_dimmer R5
 U 1 1 567D6EFA
 P 7750 2950
-F 0 "R?" V 7800 3150 50  0000 C CNN
+F 0 "R5" V 7800 3150 50  0000 C CNN
 F 1 "R" V 7750 2950 50  0000 C CNN
 F 2 "68R" V 7800 2700 50  0000 C CNN
@@
 $EndComp
 $Comp
-L R-RESCUE-led_dimmer R?
+L R-RESCUE-led_dimmer R6
 U 1 1 567D6F40
 P 7850 2950
-F 0 "R?" V 7900 3150 50  0000 C CNN
+F 0 "R6" V 7900 3150 50  0000 C CNN
 F 1 "R" V 7850 2950 50  0000 C CNN
 F 2 "68R" V 7900 2700 50  0000 C CNN
@@
 Connection ~ 7750 3100
 $Comp
-L R-RESCUE-led_dimmer R?
+L R-RESCUE-led_dimmer R7
 U 1 1 567D7788
 P 7950 2950
-F 0 "R?" V 8000 3150 50  0000 C CNN
+F 0 "R7" V 8000 3150 50  0000 C CNN
 F 1 "R" V 7950 2950 50  0000 C CNN
 F 2 "68R" V 8000 2700 50  0000 C CNN
@@
 $EndComp
 $Comp
-L R-RESCUE-led_dimmer R?
+L R-RESCUE-led_dimmer R8
 U 1 1 567D778E
 P 8050 2950
-F 0 "R?" V 8100 3150 50  0000 C CNN
+F 0 "R8" V 8100 3150 50  0000 C CNN
 F 1 "R" V 8050 2950 50  0000 C CNN
 F 2 "68R" V 8100 2700 50  0000 C CNN
@@
 $EndComp
 $Comp
-L R-RESCUE-led_dimmer R?
+L R-RESCUE-led_dimmer R9
 U 1 1 567D7794
 P 8150 2950
-F 0 "R?" V 8200 3150 50  0000 C CNN
+F 0 "R9" V 8200 3150 50  0000 C CNN
 F 1 "R" V 8150 2950 50  0000 C CNN
 F 2 "68R" V 8200 2700 50  0000 C CNN
@@
 Connection ~ 8050 3100
 $Comp
-L R-RESCUE-led_dimmer R?
+L R-RESCUE-led_dimmer R10
 U 1 1 567D780C
 P 8250 2950
-F 0 "R?" V 8300 3150 50  0000 C CNN
+F 0 "R10" V 8300 3150 50  0000 C CNN
 F 1 "R" V 8250 2950 50  0000 C CNN
 F 2 "68R" V 8300 2700 50  0000 C CNN
@@
 $EndComp
 $Comp
-L R-RESCUE-led_dimmer R?
+L R-RESCUE-led_dimmer R11
 U 1 1 567D7812
 P 8350 2950
-F 0 "R?" V 8400 3150 50  0000 C CNN
+F 0 "R11" V 8400 3150 50  0000 C CNN
 F 1 "R" V 8350 2950 50  0000 C CNN
 F 2 "68R" V 8400 2700 50  0000 C CNN
@@
 $EndComp
 $Comp
-L R-RESCUE-led_dimmer R?
+L R-RESCUE-led_dimmer R12
 U 1 1 567D7818
 P 8450 2950
-F 0 "R?" V 8500 3150 50  0000 C CNN
+F 0 "R12" V 8500 3150 50  0000 C CNN
 F 1 "R" V 8450 2950 50  0000 C CNN
 F 2 "68R" V 8500 2700 50  0000 C CNN
@@
 	7750 3250 7750 3100
 $Comp
-L CONN_4 P?
+L CONN_4 P2
 U 1 1 567D8318
 P 8100 3800
-F 0 "P?" V 8050 3800 50  0000 C CNN
+F 0 "P2" V 8050 3800 50  0000 C CNN
 F 1 "CONN_4" V 8150 3800 50  0000 C CNN
 F 2 "" H 8100 3800 60  0000 C CNN
@@
 	8450 3450 8450 4050
 $Comp
-L CONN_4 P?
+L CONN_4 P3
 U 1 1 567D8C61
 P 9100 3050
-F 0 "P?" V 9050 3050 50  0000 C CNN
+F 0 "P3" V 9050 3050 50  0000 C CNN
 F 1 "CONN_4" V 9150 3050 50  0000 C CNN
 F 2 "" H 9100 3050 60  0000 C CNN
@@
 Connection ~ 4350 2050
 $Comp
-L GND-RESCUE-led_dimmer #PWR?
+L GND-RESCUE-led_dimmer #PWR8
 U 1 1 567DBD10
 P 4600 2450
-F 0 "#PWR?" H 4600 2200 50  0001 C CNN
+F 0 "#PWR8" H 4600 2200 50  0001 C CNN
 F 1 "GND" H 4600 2300 50  0000 C CNN
 F 2 "" H 4600 2450 50  0000 C CNN
@@
 $EndComp
 $Comp
-L C C?
+L C-RESCUE-led_dimmer C4
 U 1 1 567DCE8B
 P 4600 2250
-F 0 "C?" H 4600 2350 40  0000 L CNN
+F 0 "C4" H 4600 2350 40  0000 L CNN
 F 1 "C" H 4606 2165 40  0000 L CNN
 F 2 "0.1uF" H 4700 2100 30  0000 C CNN
@@
 $EndComp
 $Comp
-L CP1 C?
+L CP1-RESCUE-led_dimmer C1
 U 1 1 567DD8B7
 P 1200 4050
-F 0 "C?" H 1250 4150 50  0000 L CNN
+F 0 "C1" H 1250 4150 50  0000 L CNN
 F 1 "CP1" H 1250 3950 50  0000 L CNN
 F 2 "10uF" H 1450 4050 60  0000 C CNN

Commit message: .
Parts:
- removed C2, C3: C, 22pF, symbol C-RESCUE-led_dimmer
- removed P2, P3: CONN_4, symbol CONN_4
- removed R11, R12, R4, R5, R6, R7: R, 68R, symbol R-RESCUE-led_dimmer
- removed X1: CRYSTAL, 8 MHz, symbol CRYSTAL
- BT1: footprint (none) -> 4.5V
Connections:
- wire segments 70 -> 46
- no-connect marks 0 -> 10
Other:
- moved on the sheet: BT1, C1, C4, C5, D1, D2, D3, IC1, P1, Q1, R1, R10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
