File: in_progress/trainer/outputs.sch (KiCad schematic (older format))
At the start: 51 parts

Commit message: .
Parts:
- D? (x16): symbol LED -> LED-RESCUE-trainer
- R? (x24): symbol R -> R-RESCUE-trainer
Changed lines of the file:
@@
 LIBS:memory
 LIBS:xilinx
-LIBS:special
 LIBS:microcontrollers
 LIBS:dsp
@@
 LIBS:valves
 LIBS:MiscellaneousDevices
+LIBS:ULN280xA
 LIBS:Gajda_cmosieee
 LIBS:jhd-162a
 LIBS:capteurs
 LIBS:trainer-cache
-EELAYER 27 0
+EELAYER 25 0
 EELAYER END
 $Descr A4 11693 8268
@@
 $EndComp
 $Comp
-L R R?
+L R-RESCUE-trainer R?
 U 1 1 565AF994
 P 9750 850
@@
 $EndComp
 $Comp
-L R R?
+L R-RESCUE-trainer R?
 U 1 1 565AF99B
 P 9750 950
@@
 $EndComp
 $Comp
-L R R?
+L R-RESCUE-trainer R?
 U 1 1 565AF9A2
 P 9750 1050
@@
 $EndComp
 $Comp
-L R R?
+L R-RESCUE-trainer R?
 U 1 1 565AF9A9
 P 9750 1150
@@
 $EndComp
 $Comp
-L R R?
+L R-RESCUE-trainer R?
 U 1 1 565AFB06
 P 9750 1250
@@
 $EndComp
 $Comp
-L R R?
+L R-RESCUE-trainer R?
 U 1 1 565AFB0C
 P 9750 1350
@@
 $EndComp
 $Comp
-L R R?
+L R-RESCUE-trainer R?
 U 1 1 565AFB12
 P 9750 1450
@@
 $EndComp
 $Comp
-L R R?
+L R-RESCUE-trainer R?
 U 1 1 565AFB18
 P 9750 1550
@@
 $EndComp
 $Comp
-L R R?
+L R-RESCUE-trainer R?
 U 1 1 565AFFED
 P 9750 2100
@@
 $EndComp
 $Comp
-L R R?
+L R-RESCUE-trainer R?
 U 1 1 565AFFF3
 P 9750 2200
@@
 $EndComp
 $Comp
-L R R?
+L R-RESCUE-trainer R?
 U 1 1 565AFFF9
 P 9750 2300
@@
 $EndComp
 $Comp
-L R R?
+L R-RESCUE-trainer R?
 U 1 1 565AFFFF
 P 9750 2400
@@
 $EndComp
 $Comp
-L R R?
+L R-RESCUE-trainer R?
 U 1 1 565B0009
 P 9750 2500
@@
 $EndComp
 $Comp
-L R R?
+L R-RESCUE-trainer R?
 U 1 1 565B000F
 P 9750 2600
@@
 $EndComp
 $Comp
-L R R?
+L R-RESCUE-trainer R?
 U 1 1 565B0015
 P 9750 2700
@@
 $EndComp
 $Comp
-L R R?
+L R-RESCUE-trainer R?
 U 1 1 565B001B
 P 9750 2800
@@
 $EndComp
 $Comp
-L LED D?
+L LED-RESCUE-trainer D?
 U 1 1 565B750A
 P 10350 850
@@
 $EndComp
 $Comp
-L LED D?
+L LED-RESCUE-trainer D?
 U 1 1 565B7969
 P 10350 950
@@
 $EndComp
 $Comp
-L LED D?
+L LED-RESCUE-trainer D?
 U 1 1 565B79BC
 P 10350 1050
@@
 $EndComp
 $Comp
-L LED D?
+L LED-RESCUE-trainer D?
 U 1 1 565B7A12
 P 10350 1150
@@
 $EndComp
 $Comp
-L LED D?
+L LED-RESCUE-trainer D?
 U 1 1 565B7A67
 P 10350 1250
@@
 $EndComp
 $Comp
-L LED D?
+L LED-RESCUE-trainer D?
 U 1 1 565B7ABF
 P 10350 1350
@@
 $EndComp
 $Comp
-L LED D?
+L LED-RESCUE-trainer D?
 U 1 1 565B7B1A
 P 10350 1450
@@
 $EndComp
 $Comp
-L LED D?
+L LED-RESCUE-trainer D?
 U 1 1 565B7B78
 P 10350 1550
@@
 $EndComp
 $Comp
-L LED D?
+L LED-RESCUE-trainer D?
 U 1 1 565B883B
 P 10350 2100
@@
 $EndComp
 $Comp
-L LED D?
+L LED-RESCUE-trainer D?
 U 1 1 565B8841
 P 10350 2200
@@
 $EndComp
 $Comp
-L LED D?
+L LED-RESCUE-trainer D?
 U 1 1 565B8847
 P 10350 2300
@@
 $EndComp
 $Comp
-L LED D?
+L LED-RESCUE-trainer D?
 U 1 1 565B884D
 P 10350 2400
@@
 $EndComp
 $Comp
-L LED D?
+L LED-RESCUE-trainer D?
 U 1 1 565B8853
 P 10350 2500
@@
 $EndComp
 $Comp
-L LED D?
+L LED-RESCUE-trainer D?
 U 1 1 565B8859
 P 10350 2600
@@
 $EndComp
 $Comp
-L LED D?
+L LED-RESCUE-trainer D?
 U 1 1 565B885F
 P 10350 2700
@@
 $EndComp
 $Comp
-L LED D?
+L LED-RESCUE-trainer D?
 U 1 1 565B8865
 P 10350 2800
@@
 $EndComp
 $Comp
-L R R?
+L R-RESCUE-trainer R?
 U 1 1 5658BCB8
 P 7200 4300
@@
 $EndComp
 $Comp
-L R R?
+L R-RESCUE-trainer R?
 U 1 1 5658C036
 P 7200 4400
@@
 $EndComp
 $Comp
-L R R?
+L R-RESCUE-trainer R?
 U 1 1 5658C0EA
 P 7200 4500
@@
 $EndComp
 $Comp
-L R R?
+L R-RESCUE-trainer R?
 U 1 1 5658C1A2
 P 7200 4600
@@
 $EndComp
 $Comp
-L R R?
+L R-RESCUE-trainer R?
 U 1 1 5659977A
 P 7200 5000
@@
 $EndComp
 $Comp
-L R R?
+L R-RESCUE-trainer R?
 U 1 1 5658C3B8
 P 7200 4900
@@
 $EndComp
 $Comp
-L R R?
+L R-RESCUE-trainer R?
 U 1 1 5658C2C7
 P 7200 4800
@@
 $EndComp
 $Comp
-L R R?
+L R-RESCUE-trainer R?
 U 1 1 5658C233
 P 7200 4700

Commit message: .
Parts:
- removed AFF?: CA56-12, symbol CA56-12
- removed IC?: ATTINY2313-P, DIP20, symbol ATTINY2313-P
- removed P?: CONN_02X08, symbol CONN_02X08
- removed R? (x8): R, 390R, symbol R-RESCUE-trainer
- removed U?: 4067, symbol 4067
- removed U?: ULN2803A, symbol ULN2803A
Connections:
- wire segments 198 -> 96
- no-connect marks 4 -> 2
Other:
- moved on the sheet: D?, P?, R?, RV?, U?

Commit message: .
Changed lines of the file:
@@
-EESchema Schematic File Version 2  date 08/12/2015 11:18:57
+EESchema Schematic File Version 2
 LIBS:trainer-rescue
 LIBS:power
@@
 LIBS:valves
 LIBS:MiscellaneousDevices
-LIBS:ULN280xA
 LIBS:Gajda_cmosieee
 LIBS:jhd-162a
 LIBS:capteurs
 LIBS:trainer-cache
-EELAYER 27 0
+EELAYER 25 0
 EELAYER END
 $Descr A4 11693 8268
@@
 	6400 4700 7050 4700
 Wire Wire Line
-	8550 2750 8850 2750
-Wire Wire Line
-	8550 2850 8850 2850
-Wire Wire Line
-	8550 2950 8850 2950
-Wire Wire Line
-	8550 3050 8850 3050
-Wire Wire Line
-	8550 3150 8850 3150
-Wire Wire Line
-	8550 3250 8850 3250
-Wire Wire Line
-	8550 3350 8850 3350
-Wire Wire Line
-	8550 3450 8850 3450
-Wire Wire Line
-	8550 4000 8850 4000
-Wire Wire Line
-	8550 4100 8850 4100
-Wire Wire Line
-	8550 4200 8850 4200
-Wire Wire Line
-	8550 4300 8850 4300
-Wire Wire Line
-	8550 4400 8850 4400
-Wire Wire Line
-	8550 4500 8850 4500
-Wire Wire Line
-	8550 4600 8850 4600
-Wire Wire Line
-	8550 4700 8850 4700
-Wire Wire Line
 	8550 3550 8600 3550
 Wire Wire Line
@@
 Connection ~ 8600 3550
 Wire Wire Line
-	9400 2750 9150 2750
-Wire Wire Line
-	9400 2850 9150 2850
-Wire Wire Line
-	9400 2950 9150 2950
-Wire Wire Line
-	9400 3050 9150 3050
-Wire Wire Line
-	9400 3150 9150 3150
-Wire Wire Line
-	9400 3250 9150 3250
-Wire Wire Line
-	9400 3350 9150 3350
-Wire Wire Line
-	9400 3450 9150 3450
-Wire Wire Line
-	9400 4000 9150 4000
-Wire Wire Line
-	9400 4100 9150 4100
-Wire Wire Line
-	9400 4200 9150 4200
-Wire Wire Line
-	9400 4300 9150 4300
-Wire Wire Line
-	9400 4400 9150 4400
-Wire Wire Line
-	9400 4500 9150 4500
-Wire Wire Line
-	9400 4600 9150 4600
-Wire Wire Line
-	9400 4700 9150 4700
-Wire Wire Line
 	9950 2750 9800 2750
 Wire Wire Line
@@
 Wire Wire Line
 	3000 3850 3000 4600
+Wire Wire Line
+	9250 3450 9400 3450
+Wire Wire Line
+	9250 3350 9400 3350
+Wire Wire Line
+	9250 3250 9400 3250
+Wire Wire Line
+	9250 3150 9400 3150
+Wire Wire Line
+	9250 3050 9400 3050
+Wire Wire Line
+	9250 2950 9400 2950
+Wire Wire Line
+	9250 2850 9400 2850
+Wire Wire Line
+	9250 2750 9400 2750
+Wire Wire Line
+	8550 3350 8750 3350
+Wire Wire Line
+	8550 3250 8750 3250
+Wire Wire Line
+	8550 3150 8750 3150
+Wire Wire Line
+	8550 3050 8750 3050
+Wire Wire Line
+	8550 2950 8750 2950
+Wire Wire Line
+	8550 2850 8750 2850
+Wire Wire Line
+	8550 2750 8750 2750
+Wire Wire Line
+	8750 3450 8550 3450
+Wire Wire Line
+	8550 4000 8750 4000
+Wire Wire Line
+	8550 4100 8750 4100
+Wire Wire Line
+	8550 4200 8750 4200
+Wire Wire Line
+	8550 4300 8750 4300
+Wire Wire Line
+	8550 4400 8750 4400
+Wire Wire Line
+	8550 4500 8750 4500
+Wire Wire Line
+	8550 4600 8750 4600
+Wire Wire Line
+	8550 4700 8750 4700
+Wire Wire Line
+	9250 4000 9400 4000
+Wire Wire Line
+	9250 4100 9400 4100
+Wire Wire Line
+	9400 4200 9250 4200
+Wire Wire Line
+	9250 4300 9400 4300
+Wire Wire Line
+	9400 4400 9250 4400
+Wire Wire Line
+	9250 4500 9400 4500
+Wire Wire Line
+	9400 4600 9250 4600
+Wire Wire Line
+	9250 4700 9400 4700
 $EndSCHEMATC
