File: in_progress/trainer/hex.sch (KiCad schematic (older format))
At the start: 16 parts

Commit message: .
Parts:
- added Q? (x4): 2N3904, TO92, symbol PN2222A
- added R? (x4): R, 1K, symbol R-RESCUE-trainer
Connections:
- wire segments 89 -> 131
- no-connect marks 2 -> 1
Other:
- note removed: "Comprar na Tiggercomp"
- note removed: "IMPORTANT: each pin should supply at most 6.5mA. \nDepending on the LEDs forward voltage, the resistors\nmust be adjusted."
- moved on the sheet: AFF?, C?, IC?, P?, R?, SP?, U?, X?

Commit message: .
Parts:
- Q? (x4): symbol PN2222A -> PN2222A-RESCUE-trainer
Connections:
- wire segments 131 -> 127
Changed lines of the file:
@@
-EESchema Schematic File Version 2  date 08/12/2015 11:18:57
+EESchema Schematic File Version 2
 LIBS:trainer-rescue
 LIBS:power
@@
 LIBS:valves
 LIBS:MiscellaneousDevices
-LIBS:ULN280xA
 LIBS:Gajda_cmosieee
 LIBS:jhd-162a
 LIBS:capteurs
 LIBS:trainer-cache
-EELAYER 27 0
+EELAYER 25 0
 EELAYER END
 $Descr A4 11693 8268
@@
 $EndComp
 $Comp
-L PN2222A Q?
+L PN2222A-RESCUE-trainer Q?
 U 1 1 5666DB86
 P 7150 3900
+AR Path="/5666DB86" Ref="Q?"  Part="1"
+AR Path="/565EDE3C/5666DB86" Ref="Q?"  Part="1"
 F 0 "Q?" H 7150 3752 40  0000 R CNN
 F 1 "2N3904" H 7150 4050 40  0000 R CNN
@@
 $EndComp
 $Comp
-L PN2222A Q?
+L PN2222A-RESCUE-trainer Q?
 U 1 1 5666DCFF
 P 7150 4400
+AR Path="/5666DCFF" Ref="Q?"  Part="1"
+AR Path="/565EDE3C/5666DCFF" Ref="Q?"  Part="1"
 F 0 "Q?" H 7150 4252 40  0000 R CNN
 F 1 "2N3904" H 7150 4550 40  0000 R CNN
@@
 $EndComp
 $Comp
-L PN2222A Q?
+L PN2222A-RESCUE-trainer Q?
 U 1 1 5666DD05
 P 7150 4900
+AR Path="/5666DD05" Ref="Q?"  Part="1"
+AR Path="/565EDE3C/5666DD05" Ref="Q?"  Part="1"
 F 0 "Q?" H 7150 4752 40  0000 R CNN
 F 1 "2N3904" H 7150 5050 40  0000 R CNN
@@
 $EndComp
 $Comp
-L PN2222A Q?
+L PN2222A-RESCUE-trainer Q?
 U 1 1 5666DD0B
 P 7150 5400
+AR Path="/5666DD0B" Ref="Q?"  Part="1"
+AR Path="/565EDE3C/5666DD0B" Ref="Q?"  Part="1"
 F 0 "Q?" H 7150 5252 40  0000 R CNN
 F 1 "2N3904" H 7150 5550 40  0000 R CNN
@@
 	3250 4200 3250 4400
 Wire Wire Line
-	4800 2050 4800 2150
-Wire Wire Line
-	4800 2150 4800 2500
+	4800 2050 4800 2500
 Wire Wire Line
 	4800 2500 3650 2500
@@
 	7250 3700 7450 3700
 Wire Wire Line
-	7450 3450 7450 3700
-Wire Wire Line
-	7450 3700 7450 4200
-Wire Wire Line
-	7450 4200 7450 4700
-Wire Wire Line
-	7450 4700 7450 5200
+	7450 3450 7450 5200
 Wire Wire Line
 	7450 4200 7250 4200

Commit message: .
Parts:
- removed C?: CP1_Small, 10nF, symbol CP1_Small
- removed IC?: ATTINY2313-P, DIP20, symbol ATTINY2313-P
- added IC?: ATMEGA16-P, DIL40, symbol ATMEGA16-P
- added RV?: POT, 10K, symbol POT
- added U?: JHD-162A, symbol JHD-162A
Connections:
- wire segments 127 -> 101
Other:
- moved on the sheet: AFF?, P?, Q?, R?, SP?, U?, X?

Commit message: .
Parts:
- removed P?: CONN_01X03, symbol CONN_01X03
- removed R? (x6): R, 390R, symbol R-RESCUE-trainer
- removed RV?: POT, 10K, symbol POT
- removed SP?: SPEAKER, symbol SPEAKER
- removed X?: Buzzer_Son, symbol Buzzer_Son
- added D?: Led_Small, symbol Led_Small
- added D? (x16): LED, symbol LED-RESCUE-trainer
- added P?: I²C, symbol CONN_01X02
- added P?: CONN_02X08, symbol CONN_02X08
- added R? (x7): R, 220R, symbol R-RESCUE-trainer
- added R?: R, 390R, symbol R-RESCUE-trainer
- added R?: R, 560R, symbol R-RESCUE-trainer
- added R? (x16): R, 330R, symbol R-RESCUE-trainer
- added RV?: POT, 10K, symbol POT
- added SW?: DEC/HEX, symbol SPST
- added U? (x2): ULN2803A, symbol ULN2803A
- R?: footprint 390R -> 220R
Connections:
- net labels added: GND
- wire segments 101 -> 270
- no-connect marks 1 -> 6
Other:
- moved on the sheet: AFF?, IC?, P?, Q?, R?, U?

Commit message: .
Parts:
- added P?: CONN_01X11, symbol CONN_01X11
Connections:
- net at IC?.19 ((OC1A)PD5), U?.5 (R/W): now also P?.2 (P2)
- net at IC?.20 ((ICP)PD6), U?.4 (RS): now also P?.1 (P1)
- net at IC?.21 ((OC2)PD7), U?.6 (E): now also P?.3 (P3)
- net at IC?.22 ((SCL)PC0), U?.14 (DB7): now also P?.11 (P11)
- net at IC?.23 ((SDA)PC1), U?.13 (DB6): now also P?.10 (P10)
- net at IC?.24 ((TCK)PC2), U?.12 (DB5): now also P?.9 (P9)
- net at IC?.25 ((TMS)PC3), U?.11 (DB4): now also P?.8 (P8)
- net at IC?.26 ((TDO)PC4), U?.10 (DB3): now also P?.7 (P7)
- net at IC?.27 ((TDI)PC5), U?.9 (DB2): now also P?.6 (P6)
- net at IC?.28 ((TOSC1)PC6), U?.8 (DB1): now also P?.5 (P5)
- net at IC?.29 ((TOSC2)PC7), U?.7 (DB0): now also P?.4 (P4)
Other:
- moved on the sheet: AFF?, D?, IC?, P?, Q?, R?, RV?, SW?, U?
