File: in_progress/trainer/hex.sch (KiCad schematic (older format))
At the start: 28 parts

Commit message: .
Parts:
- removed R?: R, 220R, symbol R-RESCUE-trainer
- added U?: ULN2803A, symbol ULN2803A
- R? (x7): footprint 220R -> 390R
- R?: footprint 1K -> 2k2
Connections:
- net GND: now also U?.9 (GND)
- net at U?.1 (Z): now also U?.14 (OUT5); no longer IC?.3 ((AIN0/INT2)PB2)
- net at U?.10 (A0): now also U?.15 (OUT4); no longer IC?.17 ((INT1)PD3)
- net at U?.11 (A1): now also U?.16 (OUT3); no longer IC?.16 ((INT0)PD2)
- net at U?.13 (A3): now also U?.17 (OUT2); no longer IC?.15 ((TXD)PD1)
- net at U?.14 (Q12): now also U?.18 (OUT1); no longer IC?.14 ((RXD)PD0)
- net at U?.4 (IN4): no longer IC?.37 ((ADC3)PA3)
- net at IC?.19 ((OC1A)PD5): now also U?.4 (RS); no longer U?.5 (R/W)
- net at IC?.20 ((ICP)PD6): now also U?.5 (R/W); no longer U?.4 (RS)
- new net: IC?.14 ((RXD)PD0), U?.1 (IN1)
- new net: IC?.15 ((TXD)PD1), U?.2 (IN2)
- new net: IC?.16 ((INT0)PD2), U?.3 (IN3)
- new net: IC?.17 ((INT1)PD3), U?.4 (IN4)
- new net: IC?.3 ((AIN0/INT2)PB2), U?.5 (IN5)
- no-connect marks 6 -> 17
Other:
- note added: "Powered by VCC"
- moved on the sheet: AFF?, D?, IC?, P?, Q?, R?, RV?, SW?, U?

Commit message: .
Parts:
- added R? (x5): R, 10k, symbol R
Connections:
- net +5V: now also R?.1
- net at U?.1 (Z): now also U?.5 (IN5); no longer U?.14 (OUT5)
- net at U?.10 (A0), U?.15 (OUT4): now also R?.2
- net at U?.11 (A1), U?.16 (OUT3): now also R?.2
- net at U?.13 (A3), U?.17 (OUT2): now also R?.2
- net at U?.14 (Q12), U?.18 (OUT1): now also R?.2
- net at IC?.3 ((AIN0/INT2)PB2): now also U?.14 (OUT5); no longer U?.5 (IN5)
- new net VCC: R?.1, R?.1, R?.1, R?.1
Other:
- moved on the sheet: P?, U?

Commit message: .
Other:
- note added: "Add pull-down resistor"
Changed lines of the file:
@@
 	1    0    0    -1
 $EndComp
+Text Notes 5350 10550 0    60   ~ 0
+Add pull-down resistor
 $EndSCHEMATC

Commit message: Liquid crystal working!
Parts:
- removed R?: R, 10k, symbol R
- R?: footprint 2k2 -> 1k8
- R? (x3): footprint 1K -> 1k8
- R?: footprint 390R -> 220R
Connections:
- net at IC?.19 ((OC1A)PD5): no longer U?.4 (RS)
- net at IC?.20 ((ICP)PD6): no longer U?.5 (R/W)
- net at IC?.21 ((OC2)PD7): no longer U?.6 (E)
- net at IC?.22 ((SCL)PC0): now also U?.4 (RS); no longer U?.14 (DB7)
- net at IC?.23 ((SDA)PC1): now also U?.5 (R/W); no longer U?.13 (DB6)
- net at IC?.24 ((TCK)PC2): now also U?.6 (E); no longer U?.12 (DB5)
- net at IC?.26 ((TDO)PC4): now also U?.12 (DB5); no longer U?.10 (DB3)
- net at IC?.27 ((TDI)PC5): now also U?.13 (DB6); no longer U?.9 (DB2)
- net at IC?.28 ((TOSC1)PC6): now also U?.14 (DB7); no longer U?.8 (DB1)
- net at IC?.29 ((TOSC2)PC7): no longer U?.7 (DB0)
- no-connect marks 17 -> 25
Other:
- moved on the sheet: D?, R?
Changed lines of the file:
@@
 F 0 "R?" V 6800 3500 50  0000 C CNN
 F 1 "R" V 6850 3300 50  0000 C CNN
-F 2 "2k2" V 6800 3100 30  0000 C CNN
+F 2 "1k8" V 6800 3100 30  0000 C CNN
 F 3 "" H 6850 3300 30  0000 C CNN
 	1    6850 3300
@@
 F 0 "R?" V 6800 3600 50  0000 C CNN
 F 1 "R" V 6850 3400 50  0000 C CNN
-F 2 "1K" V 6800 3200 30  0000 C CNN
+F 2 "1k8" V 6800 3200 30  0000 C CNN
 F 3 "" H 6850 3400 30  0000 C CNN
 	1    6850 3400
@@
 F 0 "R?" V 6800 3700 50  0000 C CNN
 F 1 "R" V 6850 3500 50  0000 C CNN
-F 2 "1K" V 6800 3300 30  0000 C CNN
+F 2 "1k8" V 6800 3300 30  0000 C CNN
 F 3 "" H 6850 3500 30  0000 C CNN
 	1    6850 3500
@@
 F 0 "R?" V 6800 3800 50  0000 C CNN
 F 1 "R" V 6850 3600 50  0000 C CNN
-F 2 "1K" V 6800 3400 30  0000 C CNN
+F 2 "1k8" V 6800 3400 30  0000 C CNN
 F 3 "" H 6850 3600 30  0000 C CNN
 	1    6850 3600
@@
 L R-RESCUE-trainer R?
 U 1 1 56687F22
-P 6050 5750
-F 0 "R?" V 6000 5950 50  0000 C CNN
-F 1 "R" V 6050 5750 50  0000 C CNN
-F 2 "390R" V 6000 5500 30  0000 C CNN
-F 3 "" H 6050 5750 30  0000 C CNN
-	1    6050 5750
+P 6150 6250
+F 0 "R?" V 6100 6450 50  0000 C CNN
+F 1 "R" V 6150 6250 50  0000 C CNN
+F 2 "220R" V 6100 6000 30  0000 C CNN
+F 3 "" H 6150 6250 30  0000 C CNN
+	1    6150 6250
 	-1   0    0    1
 $EndComp
@@
 L +5V #PWR?
 U 1 1 5668DC41
-P 6350 6100
-F 0 "#PWR?" H 6350 5950 50  0001 C CNN
-F 1 "+5V" H 6350 6240 50  0000 C CNN
-F 2 "" H 6350 6100 50  0000 C CNN
-F 3 "" H 6350 6100 50  0000 C CNN
-	1    6350 6100
+P 6450 6600
+F 0 "#PWR?" H 6450 6450 50  0001 C CNN
+F 1 "+5V" H 6450 6740 50  0000 C CNN
+F 2 "" H 6450 6600 50  0000 C CNN
+F 3 "" H 6450 6600 50  0000 C CNN
+	1    6450 6600
 	1    0    0    -1
 $EndComp
@@
 L Led_Small D?
 U 1 1 5668801F
-P 6200 6200
-F 0 "D?" H 6150 6325 50  0000 L CNN
-F 1 "Led_Small" H 6025 6100 50  0000 L CNN
-F 2 "" V 6200 6200 50  0000 C CNN
-F 3 "" V 6200 6200 50  0000 C CNN
-	1    6200 6200
+P 6300 6700
+F 0 "D?" H 6250 6825 50  0000 L CNN
+F 1 "Led_Small" H 6125 6600 50  0000 L CNN
+F 2 "" V 6300 6700 50  0000 C CNN
+F 3 "" V 6300 6700 50  0000 C CNN
+	1    6300 6700
 	1    0    0    -1
 $EndComp
@@
 	10250 4500 9400 4500
 Wire Wire Line
-	6350 6100 6350 6200
-Wire Wire Line
-	6350 6200 6300 6200
-Wire Wire Line
-	5450 5100 6050 5100
-Wire Wire Line
-	6050 5100 6050 5500
-Wire Wire Line
-	6050 6000 6050 6200
-Wire Wire Line
-	6050 6200 6100 6200
-Wire Wire Line
-	5450 3800 7000 3800
-Wire Wire Line
-	7000 3800 7000 5550
-Wire Wire Line
-	7000 5550 10050 5550
-Wire Wire Line
-	5450 3900 6950 3900
-Wire Wire Line
-	6950 3900 6950 5650
-Wire Wire Line
-	6950 5650 10050 5650
-Wire Wire Line
-	5450 4000 6900 4000
-Wire Wire Line
-	6900 4000 6900 5750
-Wire Wire Line
-	6900 5750 10050 5750
-Wire Wire Line
-	5450 4100 6850 4100
-Wire Wire Line
-	6850 4100 6850 5850
-Wire Wire Line
-	6850 5850 10050 5850
-Wire Wire Line
-	5450 4200 6800 4200
-Wire Wire Line
-	6800 4200 6800 5950
-Wire Wire Line
-	6800 5950 10050 5950
-Wire Wire Line
-	5450 4300 6750 4300
-Wire Wire Line
-	6750 4300 6750 6050
-Wire Wire Line
-	6750 6050 10050 6050
-Wire Wire Line
-	5450 4400 6700 4400
-Wire Wire Line
-	6700 4400 6700 6150
-Wire Wire Line
-	6700 6150 10050 6150
-Wire Wire Line
-	5450 4500 6650 4500
-Wire Wire Line
-	6650 4500 6650 6250
-Wire Wire Line
-	6650 6250 10050 6250
-Wire Wire Line
-	5450 5400 6600 5400
-Wire Wire Line
-	6600 5400 6600 6350
-Wire Wire Line
-	6600 6350 10050 6350
+	6450 6600 6450 6700
+Wire Wire Line
+	6450 6700 6400 6700
+Wire Wire Line
+	5450 5100 6150 5100
+Wire Wire Line
+	6150 5100 6150 6000
+Wire Wire Line
+	6150 6500 6150 6700
+Wire Wire Line
+	6150 6700 6200 6700
 Wire Wire Line
 	9550 6750 10050 6750
@@
 Wire Wire Line
 	6050 8300 6050 8100
-Wire Wire Line
-	5450 5200 6550 5200
-Wire Wire Line
-	6550 5200 6550 6550
-Wire Wire Line
-	6550 6550 10050 6550
-Wire Wire Line
-	5450 5300 6500 5300
-Wire Wire Line
-	6500 5300 6500 6450
-Wire Wire Line
-	6500 6450 10050 6450
 Wire Wire Line
 	5450 2000 6100 2000
@@
 Wire Wire Line
 	5450 3100 5500 3100
-$Comp
-L R R?
-U 1 1 566C1523
-P 5500 1650
-F 0 "R?" V 5580 1650 50  0000 C CNN
-F 1 "R" V 5500 1650 50  0000 C CNN
-F 2 "10k" V 5430 1650 50  0000 C CNN
-F 3 "" H 5500 1650 50  0000 C CNN
-	1    5500 1650
-	1    0    0    -1
-$EndComp
-$Comp
-L +5V #PWR?
-U 1 1 566C1605
-P 5500 1500
-F 0 "#PWR?" H 5500 1350 50  0001 C CNN
-F 1 "+5V" H 5500 1640 50  0000 C CNN
-F 2 "" H 5500 1500 50  0000 C CNN
-F 3 "" H 5500 1500 50  0000 C CNN
-	1    5500 1500
-	1    0    0    -1
-$EndComp
 Wire Wire Line
 	5500 7000 7700 7000
@@
 	5800 7700 6050 7700
 Wire Wire Line
-	6050 7300 5550 7300
-Wire Wire Line
-	5550 7300 5550 4700
-Wire Wire Line
-	5550 4700 5450 4700
-Wire Wire Line
-	6050 7400 5600 7400
-Wire Wire Line
-	5600 7400 5600 4800
-Wire Wire Line
-	5600 4800 5450 4800
-Wire Wire Line
-	6050 7500 5650 7500
-Wire Wire Line
-	5650 7500 5650 4900
-Wire Wire Line
-	5650 4900 5450 4900
-Wire Wire Line
-	6050 7600 5700 7600
-Wire Wire Line
-	5700 7600 5700 5000
-Wire Wire Line
-	5700 5000 5450 5000
+	6050 7300 5600 7300
+Wire Wire Line
+	5600 7300 5600 4700
+Wire Wire Line
+	5600 4700 5450 4700
+Wire Wire Line
+	6050 7400 5700 7400
+Wire Wire Line
+	5700 7400 5700 4800
+Wire Wire Line
+	5700 4800 5450 4800
+Wire Wire Line
+	6050 7500 5800 7500
+Wire Wire Line
+	5800 7500 5800 4900
+Wire Wire Line
+	5800 4900 5450 4900
+Wire Wire Line
+	6050 7600 5900 7600
+Wire Wire Line
+	5900 7600 5900 5000
+Wire Wire Line
+	5900 5000 5450 5000
 Wire Wire Line
 	7900 9500 7550 9500
@@
 Text Notes 5350 10550 0    60   ~ 0
 Add pull-down resistor
+Wire Wire Line
+	5450 3800 6900 3800
+Wire Wire Line
+	6900 3800 6900 6550
+Wire Wire Line
+	6900 6550 10050 6550
+Wire Wire Line
+	5450 3900 6800 3900
+Wire Wire Line
+	6800 3900 6800 6450
+Wire Wire Line
+	6800 6450 10050 6450
+Wire Wire Line
+	5450 4000 6700 4000
+Wire Wire Line
+	6700 4000 6700 6350
+Wire Wire Line
+	6700 6350 10050 6350
+Wire Wire Line
+	5450 4100 6600 4100
+Wire Wire Line
+	6600 4100 6600 5850
+Wire Wire Line
+	6600 5850 10050 5850
+Wire Wire Line
+	5450 4200 6500 4200
+Wire Wire Line
+	6500 4200 6500 5750
+Wire Wire Line
+	6500 5750 10050 5750
+Wire Wire Line
+	5450 4300 6400 4300
+Wire Wire Line
+	6400 4300 6400 5650
+Wire Wire Line
+	6400 5650 10050 5650
+Wire Wire Line
+	5450 4400 6300 4400
+Wire Wire Line
+	6300 4400 6300 5550
+Wire Wire Line
+	6300 5550 10050 5550
+NoConn ~ 5450 4500
+NoConn ~ 5450 5200
+NoConn ~ 5450 5300
+NoConn ~ 5450 5400
+NoConn ~ 10050 5950
+NoConn ~ 10050 6050
+NoConn ~ 10050 6150
+NoConn ~ 10050 6250
 $EndSCHEMATC

Commit message: .
Parts:
- removed P?: I²C, symbol CONN_01X02
Connections:
- no-connect marks 25 -> 27
Changed lines of the file:
@@
-$EndComp
-$Comp
-L CONN_01X02 P?
-U 1 1 566825DC
-P 5850 2950
-F 0 "P?" H 5850 3100 50  0000 C CNN
-F 1 "I²C" V 5950 2950 50  0000 C CNN
-F 2 "" H 5850 2950 50  0000 C CNN
-F 3 "" H 5850 2950 50  0000 C CNN
-	1    5850 2950
-	1    0    0    -1
 $EndComp
 $Comp
@@
 $EndComp
 Wire Wire Line
-	5450 2900 5650 2900
-Wire Wire Line
-	5450 3000 5650 3000
-Wire Wire Line
 	5450 3100 5500 3100
 Wire Wire Line
@@
 NoConn ~ 10050 6150
 NoConn ~ 10050 6250
+NoConn ~ 5450 3000
+NoConn ~ 5450 2900
 $EndSCHEMATC

Commit message: .
Parts:
- removed R? (x4): R, 10k, symbol R
- removed U?: ULN2803A, symbol ULN2803A
- added R? (x16): R, 10k, symbol R
Connections:
- net GND: now also R?.1, R?.1, R?.1, R?.1, R?.1, R?.1, R?.1, R?.1, R?.1, R?.1, R?.1, R?.1, R?.1, R?.1, R?.1, R?.1
- net at U?.1 (Z): now also IC?.3 ((AIN0/INT2)PB2)
- net at U?.10 (A0): now also IC?.17 ((INT1)PD3)
- net at U?.11 (A1): now also IC?.16 ((INT0)PD2)
- net at U?.13 (A3): now also IC?.4 ((AIN1/OC0)PB3)
- net at P?.10 (P10), U?.14 (Q12): now also R?.2
- net at U?.14 (Q12): now also IC?.2 ((T1)PB1)
- net at P?.16 (P16), U?.17 (A15): now also R?.2
- net at P?.14 (P14), U?.18 (A14): now also R?.2
- net at P?.12 (P12), U?.19 (A13): now also R?.2
- net at P?.15 (P15), U?.2 (A7): now also R?.2
- net at P?.8 (P8), U?.20 (A11): now also R?.2
- net at P?.6 (P6), U?.21 (A10): now also R?.2
- net at P?.4 (P4), U?.22 (A9): now also R?.2
- net at P?.2 (P2), U?.23 (A8): now also R?.2
- net at P?.13 (P13), U?.3 (A3): now also R?.2
- net at P?.11 (P11), U?.4 (A5): now also R?.2
- net at P?.9 (P9), U?.5 (A4): now also R?.2
- net at P?.7 (P7), U?.6 (A3): now also R?.2
- net at P?.5 (P5), U?.7 (A2): now also R?.2
- net at P?.3 (P3), U?.8 (A1): now also R?.2
- net at P?.1 (P1), U?.9 (A0): now also R?.2
- net at R?.2: now also IC?.18 ((OC1B)PD4); no longer IC?.5 ((~SS~)PB4)
- net at R?.2: now also IC?.19 ((OC1A)PD5); no longer IC?.6 ((MOSI)PB5)
- net at R?.2: now also IC?.20 ((ICP)PD6); no longer IC?.7 ((MISO)PB6)
- net at R?.2: now also IC?.21 ((OC2)PD7); no longer IC?.8 ((SCK)PB7)
- net at R?.2: now also IC?.29 ((TOSC2)PC7); no longer IC?.18 ((OC1B)PD4)
- net at IC?.37 ((ADC3)PA3): now also SW?.1
- no-connect marks 27 -> 18
Other:
- note removed: "Add pull-down resistor"
- moved on the sheet: AFF?, D?, IC?, P?, Q?, R?, RV?, SW?, U?

Commit message: .
Parts:
- added P?: CONN_01X02, UART, symbol CONN_01X02
- R?: footprint 220R -> 560R
Connections:
- net at IC?.14 ((RXD)PD0): now also P?.1 (P1)
- net at IC?.15 ((TXD)PD1): now also P?.2 (P2)
Other:
- moved on the sheet: AFF?, D?, IC?, P?, Q?, R?, RV?, SW?, U?

Commit message: .
Parts:
- added SW23: SW_PUSH, SCRL_UP, symbol SW_PUSH
- added SW24: SW_PUSH, SCRL_DOWN, symbol SW_PUSH
- gave numbers to parts that had none: 43
Connections:
- net GND: now also SW23.2, SW24.2
- net at IC1.1 ((T0/XCK)PB0): now also SW23.1
- net at IC1.5 ((~SS~)PB4): now also SW24.1
- no-connect marks 18 -> 16
