File: in_progress/trainer/hex.sch (KiCad schematic (older format))
At the start: 45 parts, among them IC1 ATMEGA16-P, P12 CONN_02X08, P13 CONN_01X02, Q2 2N3904, Q3 2N3904, Q4 2N3904, Q5 2N3904, SW22 DEC/HEX, SW23 SW_PUSH, SW24 SW_PUSH, U10 JHD-162A, U8 4067, U9 ULN2803A

Commit message: .
Parts:
- removed D17: Led_Small, symbol Led_Small
- removed R43: R, 560R, symbol R-RESCUE-trainer
- added D?: Led_Small, symbol Led_Small
- added R?: R, 560R, symbol R
Connections:
- net GND: now also D?.1 (K)
- net at U8.10 (A0): now also IC1.5 ((~SS~)PB4); no longer IC1.17 ((INT1)PD3)
- net at U8.11 (A1): now also IC1.1 ((T0/XCK)PB0); no longer IC1.16 ((INT0)PD2)
- net at SW23.1: now also IC1.16 ((INT0)PD2); no longer IC1.1 ((T0/XCK)PB0)
- net at IC1.29 ((TOSC2)PC7): now also R?.2
- net at SW24.1: now also IC1.17 ((INT1)PD3); no longer IC1.5 ((~SS~)PB4)
- new net: D?.2 (A), R?.1
Other:
- moved on the sheet: P13, SW23, SW24
Changed lines of the file:
@@
-$EndComp
-$Comp
-L R-RESCUE-trainer R43
-U 1 1 56687F22
-P 7350 6700
-F 0 "R43" V 7300 6900 50  0000 C CNN
-F 1 "R" V 7350 6700 50  0000 C CNN
-F 2 "560R" V 7300 6450 30  0000 C CNN
-F 3 "" H 7350 6700 30  0000 C CNN
-	1    7350 6700
-	-1   0    0    1
-$EndComp
-$Comp
-L +5V #PWR62
-U 1 1 5668DC41
-P 7650 7050
-F 0 "#PWR62" H 7650 6900 50  0001 C CNN
-F 1 "+5V" H 7650 7190 50  0000 C CNN
-F 2 "" H 7650 7050 50  0000 C CNN
-F 3 "" H 7650 7050 50  0000 C CNN
-	1    7650 7050
-	1    0    0    -1
-$EndComp
-$Comp
-L Led_Small D17
-U 1 1 5668801F
-P 7500 7150
-F 0 "D17" H 7450 7275 50  0000 L CNN
-F 1 "Led_Small" H 7325 7050 50  0000 L CNN
-F 2 "" V 7500 7150 50  0000 C CNN
-F 3 "" V 7500 7150 50  0000 C CNN
-	1    7500 7150
-	1    0    0    -1
 $EndComp
 $Comp
@@
 L CONN_01X02 P13
 U 1 1 5669A8F7
-P 7100 5200
-F 0 "P13" H 7100 5350 50  0000 C CNN
-F 1 "CONN_01X02" V 7200 5200 50  0000 C CNN
-F 2 "UART" H 7050 5050 50  0000 C CNN
-F 3 "" H 7100 5200 50  0000 C CNN
-	1    7100 5200
+P 8400 5200
+F 0 "P13" H 8400 5350 50  0000 C CNN
+F 1 "CONN_01X02" V 8500 5200 50  0000 C CNN
+F 2 "UART" H 8350 5050 50  0000 C CNN
+F 3 "" H 8400 5200 50  0000 C CNN
+	1    8400 5200
 	1    0    0    -1
 $EndComp
@@
 L SW_PUSH SW23
 U 1 1 566A89D8
-P 7700 3700
-F 0 "SW23" H 7850 3810 50  0000 C CNN
-F 1 "SW_PUSH" H 7700 3620 50  0000 C CNN
-F 2 "SCRL_UP" H 7350 3750 50  0000 C CNN
-F 3 "" H 7700 3700 50  0000 C CNN
-	1    7700 3700
+P 8200 7500
+F 0 "SW23" H 8350 7610 50  0000 C CNN
+F 1 "SW_PUSH" H 8200 7420 50  0000 C CNN
+F 2 "SCRL_UP" H 7850 7550 50  0000 C CNN
+F 3 "" H 8200 7500 50  0000 C CNN
+	1    8200 7500
 	1    0    0    -1
 $EndComp
@@
 L SW_PUSH SW24
 U 1 1 566A8AAD
-P 7700 4000
-F 0 "SW24" H 7850 4110 50  0000 C CNN
-F 1 "SW_PUSH" H 7700 3920 50  0000 C CNN
-F 2 "SCRL_DOWN" H 7300 4050 50  0000 C CNN
-F 3 "" H 7700 4000 50  0000 C CNN
-	1    7700 4000
+P 8200 7800
+F 0 "SW24" H 8350 7910 50  0000 C CNN
+F 1 "SW_PUSH" H 8200 7720 50  0000 C CNN
+F 2 "SCRL_DOWN" H 7800 7850 50  0000 C CNN
+F 3 "" H 8200 7800 50  0000 C CNN
+	1    8200 7800
 	1    0    0    -1
 $EndComp
@@
 L GND #PWR64
 U 1 1 566A8FFF
-P 8050 4050
-F 0 "#PWR64" H 8050 3800 50  0001 C CNN
-F 1 "GND" H 8050 3900 50  0000 C CNN
-F 2 "" H 8050 4050 50  0000 C CNN
-F 3 "" H 8050 4050 50  0000 C CNN
-	1    8050 4050
+P 8550 7850
+F 0 "#PWR64" H 8550 7600 50  0001 C CNN
+F 1 "GND" H 8550 7700 50  0000 C CNN
+F 2 "" H 8550 7850 50  0000 C CNN
+F 3 "" H 8550 7850 50  0000 C CNN
+	1    8550 7850
 	1    0    0    -1
 $EndComp
@@
 	12200 4950 11350 4950
 Wire Wire Line
-	7650 7050 7650 7150
-Wire Wire Line
-	7650 7150 7600 7150
-Wire Wire Line
-	7350 4950 7350 6450
-Wire Wire Line
-	7350 6950 7350 7150
-Wire Wire Line
-	7350 7150 7400 7150
-Wire Wire Line
 	11600 7200 12100 7200
 Wire Wire Line
@@
 	6600 3550 6650 3550
 Wire Wire Line
-	6950 5350 6600 5350
-Wire Wire Line
-	7050 5450 6600 5450
-Wire Wire Line
 	6750 7300 6250 7300
 Wire Wire Line
 	6850 7200 6250 7200
 Wire Wire Line
-	6250 7400 6950 7400
-Wire Wire Line
-	6250 7500 7050 7500
+	6950 7400 6250 7400
+Wire Wire Line
+	7050 7500 6250 7500
 Wire Wire Line
 	6600 4250 8050 4250
@@
 	6650 6800 6250 6800
 Wire Wire Line
-	7050 7500 7050 5450
-Wire Wire Line
-	6950 7400 6950 5350
+	7050 3750 7050 7500
+Wire Wire Line
+	6950 3350 6950 7400
 Wire Wire Line
 	6750 3450 6750 7300
@@
 	6600 3650 6850 3650
 Wire Wire Line
-	6600 5150 6900 5150
-Wire Wire Line
-	6600 5250 6900 5250
+	6600 5150 8200 5150
+Wire Wire Line
+	6600 5250 8200 5250
 Wire Wire Line
 	6600 5550 8150 5550
@@
 	6650 3550 6650 6800
 Wire Wire Line
-	6600 3350 6950 3350
-Wire Wire Line
-	6950 3350 6950 3700
-Wire Wire Line
-	6950 3700 7400 3700
-Wire Wire Line
-	6600 3750 6950 3750
-Wire Wire Line
-	6950 3750 6950 4000
-Wire Wire Line
-	6950 4000 7400 4000
-Wire Wire Line
-	8000 4000 8050 4000
-Wire Wire Line
-	8050 3700 8050 4050
-Wire Wire Line
-	8000 3700 8050 3700
-Connection ~ 8050 4000
+	8500 7800 8550 7800
+Wire Wire Line
+	8550 7500 8550 7850
+Wire Wire Line
+	8500 7500 8550 7500
+Connection ~ 8550 7800
+Wire Wire Line
+	6950 3350 6600 3350
+Wire Wire Line
+	7050 3750 6600 3750
+$Comp
+L R R?
+U 1 1 568B24E5
+P 7500 3950
+F 0 "R?" V 7580 3950 50  0000 C CNN
+F 1 "R" V 7500 3950 50  0000 C CNN
+F 2 "560R" V 7430 3950 50  0000 C CNN
+F 3 "" H 7500 3950 50  0000 C CNN
+	1    7500 3950
+	0    1    1    0
+$EndComp
+$Comp
+L Led_Small D?
+U 1 1 568B300A
+P 7900 3950
+F 0 "D?" H 7850 4075 50  0000 L CNN
+F 1 "Led_Small" H 7725 3850 50  0000 L CNN
+F 2 "" V 7900 3950 50  0000 C CNN
+F 3 "" V 7900 3950 50  0000 C CNN
+	1    7900 3950
+	-1   0    0    1
+$EndComp
+$Comp
+L GND #PWR?
+U 1 1 568B30CE
+P 8100 4000
+F 0 "#PWR?" H 8100 3750 50  0001 C CNN
+F 1 "GND" H 8100 3850 50  0000 C CNN
+F 2 "" H 8100 4000 50  0000 C CNN
+F 3 "" H 8100 4000 50  0000 C CNN
+	1    8100 4000
+	1    0    0    -1
+$EndComp
+Wire Wire Line
+	8100 4000 8100 3950
+Wire Wire Line
+	8100 3950 8000 3950
+Wire Wire Line
+	7350 4950 7350 3950
+Wire Wire Line
+	7650 3950 7800 3950
+Wire Wire Line
+	6600 5350 7200 5350
+Wire Wire Line
+	7200 5350 7200 7500
+Wire Wire Line
+	7200 7500 7900 7500
+Wire Wire Line
+	6600 5450 7300 5450
+Wire Wire Line
+	7300 5450 7300 7800
+Wire Wire Line
+	7300 7800 7900 7800
 $EndSCHEMATC

Commit message: Digital block done!
Parts:
- added C?: C, 0.1uF, symbol C
Connections:
- net +5V: now also C?.1
- net GND: now also C?.2
Changed lines of the file:
@@
 L GND #PWR59
 U 1 1 5667DC7C
-P 5550 6150
-F 0 "#PWR59" H 5550 5900 50  0001 C CNN
-F 1 "GND" H 5550 6000 50  0000 C CNN
-F 2 "" H 5550 6150 50  0000 C CNN
-F 3 "" H 5550 6150 50  0000 C CNN
-	1    5550 6150
+P 5550 6250
+F 0 "#PWR59" H 5550 6000 50  0001 C CNN
+F 1 "GND" H 5550 6100 50  0000 C CNN
+F 2 "" H 5550 6250 50  0000 C CNN
+F 3 "" H 5550 6250 50  0000 C CNN
+	1    5550 6250
 	1    0    0    -1
 $EndComp
@@
 Wire Wire Line
 	7300 7800 7900 7800
+$Comp
+L C C?
+U 1 1 568DF9AB
+P 4200 2700
+F 0 "C?" H 4225 2800 50  0000 L CNN
+F 1 "C" H 4225 2600 50  0000 L CNN
+F 2 "0.1uF" H 4050 2600 50  0000 C CNN
+F 3 "" H 4200 2700 50  0000 C CNN
+	1    4200 2700
+	1    0    0    -1
+$EndComp
+Wire Wire Line
+	5550 6250 5550 6150
+Wire Wire Line
+	5550 6200 4200 6200
+Wire Wire Line
+	4200 6200 4200 2850
+Connection ~ 5550 6200
+Wire Wire Line
+	4200 2550 4200 2050
+Wire Wire Line
+	4200 2050 5450 2050
+Connection ~ 5450 2050
 $EndSCHEMATC

Commit message: .
Parts:
- removed R44, R45, R46, R47: R, 1k8, symbol R-RESCUE-trainer
- added R? (x4): R, 1k8, symbol R
- added R? (x2): R, 10k, symbol R
Connections:
- net GND: now also R?.2, R?.2
- net at Q2.2 (B): now also R?.1
- net at IC1.18 ((OC1B)PD4): now also R?.2
- net at Q3.2 (B): now also R?.1
- net at IC1.19 ((OC1A)PD5): now also R?.2
- net at Q4.2 (B): now also R?.1
- net at IC1.20 ((ICP)PD6): now also R?.2
- net at Q5.2 (B): now also R?.1
- net at IC1.21 ((OC2)PD7): now also R?.2
- net at IC1.14 ((RXD)PD0), P13.1 (P1): now also R?.1
- net at IC1.15 ((TXD)PD1), P13.2 (P2): now also R?.1
Other:
- moved on the sheet: D?, P13, R?
Changed lines of the file:
@@
-$EndComp
-$Comp
-L R-RESCUE-trainer R44
-U 1 1 5666DBF2
-P 8400 5550
-F 0 "R44" V 8350 5750 50  0000 C CNN
-F 1 "R" V 8400 5550 50  0000 C CNN
-F 2 "1k8" V 8350 5350 30  0000 C CNN
-F 3 "" H 8400 5550 30  0000 C CNN
-	1    8400 5550
-	0    1    1    0
-$EndComp
-$Comp
-L R-RESCUE-trainer R45
-U 1 1 5666DC11
-P 8400 5650
-F 0 "R45" V 8350 5850 50  0000 C CNN
-F 1 "R" V 8400 5650 50  0000 C CNN
-F 2 "1k8" V 8350 5450 30  0000 C CNN
-F 3 "" H 8400 5650 30  0000 C CNN
-	1    8400 5650
-	0    1    1    0
-$EndComp
-$Comp
-L R-RESCUE-trainer R46
-U 1 1 5666DC17
-P 8400 5750
-F 0 "R46" V 8350 5950 50  0000 C CNN
-F 1 "R" V 8400 5750 50  0000 C CNN
-F 2 "1k8" V 8350 5550 30  0000 C CNN
-F 3 "" H 8400 5750 30  0000 C CNN
-	1    8400 5750
-	0    1    1    0
-$EndComp
-$Comp
-L R-RESCUE-trainer R47
-U 1 1 5666DC1D
-P 8400 5850
-F 0 "R47" V 8350 6050 50  0000 C CNN
-F 1 "R" V 8400 5850 50  0000 C CNN
-F 2 "1k8" V 8350 5650 30  0000 C CNN
-F 3 "" H 8400 5850 30  0000 C CNN
-	1    8400 5850
-	0    1    1    0
 $EndComp
 $Comp
@@
 L CONN_01X02 P13
 U 1 1 5669A8F7
-P 8400 5200
-F 0 "P13" H 8400 5350 50  0000 C CNN
-F 1 "CONN_01X02" V 8500 5200 50  0000 C CNN
-F 2 "UART" H 8350 5050 50  0000 C CNN
-F 3 "" H 8400 5200 50  0000 C CNN
-	1    8400 5200
+P 8300 3750
+F 0 "P13" H 8300 3900 50  0000 C CNN
+F 1 "CONN_01X02" V 8400 3750 50  0000 C CNN
+F 2 "UART" H 8250 3600 50  0000 C CNN
+F 3 "" H 8300 3750 50  0000 C CNN
+	1    8300 3750
 	1    0    0    -1
 $EndComp
@@
 	7450 6000 12100 6000
 Wire Wire Line
-	6600 4950 7350 4950
+	6600 4950 8050 4950
 Wire Wire Line
 	9400 3150 12200 3150
@@
 	6600 3650 6850 3650
 Wire Wire Line
-	6600 5150 8200 5150
-Wire Wire Line
-	6600 5250 8200 5250
-Wire Wire Line
-	6600 5550 8150 5550
-Wire Wire Line
-	6600 5650 8150 5650
-Wire Wire Line
-	6600 5750 8150 5750
-Wire Wire Line
-	6600 5850 8150 5850
+	6600 5550 8350 5550
+Wire Wire Line
+	6600 5650 8350 5650
+Wire Wire Line
+	6600 5750 8350 5750
+Wire Wire Line
+	6600 5850 8350 5850
 Wire Wire Line
 	8650 5550 8650 3750
@@
 L R R?
 U 1 1 568B24E5
-P 7500 3950
-F 0 "R?" V 7580 3950 50  0000 C CNN
-F 1 "R" V 7500 3950 50  0000 C CNN
-F 2 "560R" V 7430 3950 50  0000 C CNN
-F 3 "" H 7500 3950 50  0000 C CNN
-	1    7500 3950
+P 8200 4950
+F 0 "R?" V 8280 4950 50  0000 C CNN
+F 1 "R" V 8200 4950 50  0000 C CNN
+F 2 "560R" V 8130 4950 50  0000 C CNN
+F 3 "" H 8200 4950 50  0000 C CNN
+	1    8200 4950
 	0    1    1    0
 $EndComp
@@
 L Led_Small D?
 U 1 1 568B300A
-P 7900 3950
-F 0 "D?" H 7850 4075 50  0000 L CNN
-F 1 "Led_Small" H 7725 3850 50  0000 L CNN
-F 2 "" V 7900 3950 50  0000 C CNN
-F 3 "" V 7900 3950 50  0000 C CNN
-	1    7900 3950
+P 8450 4950
+F 0 "D?" H 8400 5075 50  0000 L CNN
+F 1 "Led_Small" H 8150 4850 50  0000 L CNN
+F 2 "" V 8450 4950 50  0000 C CNN
+F 3 "" V 8450 4950 50  0000 C CNN
+	1    8450 4950
 	-1   0    0    1
 $EndComp
@@
 L GND #PWR?
 U 1 1 568B30CE
-P 8100 4000
-F 0 "#PWR?" H 8100 3750 50  0001 C CNN
-F 1 "GND" H 8100 3850 50  0000 C CNN
-F 2 "" H 8100 4000 50  0000 C CNN
-F 3 "" H 8100 4000 50  0000 C CNN
-	1    8100 4000
-	1    0    0    -1
-$EndComp
-Wire Wire Line
-	8100 4000 8100 3950
-Wire Wire Line
-	8100 3950 8000 3950
-Wire Wire Line
-	7350 4950 7350 3950
-Wire Wire Line
-	7650 3950 7800 3950
+P 8550 5000
+F 0 "#PWR?" H 8550 4750 50  0001 C CNN
+F 1 "GND" H 8550 4850 50  0000 C CNN
+F 2 "" H 8550 5000 50  0000 C CNN
+F 3 "" H 8550 5000 50  0000 C CNN
+	1    8550 5000
+	1    0    0    -1
+$EndComp
+Wire Wire Line
+	8550 4950 8550 5000
+Wire Wire Line
+	8350 4950 8350 4950
 Wire Wire Line
 	6600 5350 7200 5350
@@
 $EndComp
 Wire Wire Line
-	5550 6250 5550 6150
+	5550 6150 5550 6250
 Wire Wire Line
 	5550 6200 4200 6200
@@
 	4200 2050 5450 2050
 Connection ~ 5450 2050
+$Comp
+L R R?
+U 1 1 568E36BE
+P 8500 5550
+F 0 "R?" V 8450 5750 50  0000 C CNN
+F 1 "R" V 8500 5550 50  0000 C CNN
+F 2 "1k8" V 8450 5350 50  0000 C CNN
+F 3 "" H 8500 5550 50  0000 C CNN
+	1    8500 5550
+	0    1    1    0
+$EndComp
+$Comp
+L R R?
+U 1 1 568E393C
+P 8500 5650
+F 0 "R?" V 8450 5850 50  0000 C CNN
+F 1 "R" V 8500 5650 50  0000 C CNN
+F 2 "1k8" V 8450 5450 50  0000 C CNN
+F 3 "" H 8500 5650 50  0000 C CNN
+	1    8500 5650
+	0    1    1    0
+$EndComp
+$Comp
+L R R?
+U 1 1 568E39D0
+P 8500 5750
+F 0 "R?" V 8450 5950 50  0000 C CNN
+F 1 "R" V 8500 5750 50  0000 C CNN
+F 2 "1k8" V 8450 5550 50  0000 C CNN
+F 3 "" H 8500 5750 50  0000 C CNN
+	1    8500 5750
+	0    1    1    0
+$EndComp
+$Comp
+L R R?
+U 1 1 568E3A67
+P 8500 5850
+F 0 "R?" V 8450 6050 50  0000 C CNN
+F 1 "R" V 8500 5850 50  0000 C CNN
+F 2 "1k8" V 8450 5650 50  0000 C CNN
+F 3 "" H 8500 5850 50  0000 C CNN
+	1    8500 5850
+	0    1    1    0
+$EndComp
+Wire Wire Line
+	6600 5150 7200 5150
+Wire Wire Line
+	7200 5150 7200 3700
+Wire Wire Line
+	7200 3700 8100 3700
+Wire Wire Line
+	6600 5250 7300 5250
+Wire Wire Line
+	7300 5250 7300 3800
+Wire Wire Line
+	7300 3800 8100 3800
+$Comp
+L R R?
+U 1 1 568E50BC
+P 7750 4000
+F 0 "R?" V 7830 4000 50  0000 C CNN
+F 1 "R" V 7750 4000 50  0000 C CNN
+F 2 "10k" V 7680 4000 50  0000 C CNN
+F 3 "" H 7750 4000 50  0000 C CNN
+	1    7750 4000
+	1    0    0    -1
+$EndComp
+$Comp
+L R R?
+U 1 1 568E51CB
+P 8000 4000
+F 0 "R?" V 8080 4000 50  0000 C CNN
+F 1 "R" V 8000 4000 50  0000 C CNN
+F 2 "10k" V 7930 4000 50  0000 C CNN
+F 3 "" H 8000 4000 50  0000 C CNN
+	1    8000 4000
+	1    0    0    -1
+$EndComp
+$Comp
+L GND #PWR?
+U 1 1 568E5271
+P 7750 4150
+F 0 "#PWR?" H 7750 3900 50  0001 C CNN
+F 1 "GND" H 7750 4000 50  0000 C CNN
+F 2 "" H 7750 4150 50  0000 C CNN
+F 3 "" H 7750 4150 50  0000 C CNN
+	1    7750 4150
+	1    0    0    -1
+$EndComp
+$Comp
+L GND #PWR?
+U 1 1 568E530C
+P 8000 4150
+F 0 "#PWR?" H 8000 3900 50  0001 C CNN
+F 1 "GND" H 8000 4000 50  0000 C CNN
+F 2 "" H 8000 4150 50  0000 C CNN
+F 3 "" H 8000 4150 50  0000 C CNN
+	1    8000 4150
+	1    0    0    -1
+$EndComp
+Wire Wire Line
+	7750 3850 7750 3700
+Connection ~ 7750 3700
+Wire Wire Line
+	8000 3850 8000 3800
+Connection ~ 8000 3800
 $EndSCHEMATC

Commit message: .
Parts:
- gave numbers to parts that had none: 9
- renumbered P12 to P13, P13 to P14, Q2 to Q3, Q3 to Q4, Q4 to Q5, Q5 to Q6, R27 to R23, R28 to R24, R29 to R25, R30 to R26, R31 to R27, R32 to R28, R33 to R29, R34 to R30, R35 to R31, R36 to R32, R37 to R33, R38 to R34, R39 to R35, R40 to R36, R41 to R37, R42 to R38, R48 to R46, R49 to R47, R50 to R48, R51 to R49, R52 to R50, R53 to R51, R54 to R52, R55 to R53, SW22 to SW21, SW23 to SW22, SW24 to SW23, U8 to U6, U9 to U7, U10 to U8

Commit message: .
Parts:
- added C12: C, 0.1uF, symbol C
- renumbered P14 to P10, P13 to P9, U6 to U7, U7 to U8, U8 to U9
Connections:
- net GND: now also C12.2
- new net VCC: C12.1
Other:
- note removed: "Powered by VCC"
Changed lines of the file:
@@
 $EndDescr
 $Comp
-L CONN_02X08 P13
+L CONN_02X08 P9
 U 1 1 565EE936
 P 3050 7750
-F 0 "P13" H 3050 8200 50  0000 C CNN
+F 0 "P9" H 3050 8200 50  0000 C CNN
 F 1 "CONN_02X08" V 3050 7750 50  0000 C CNN
 F 2 "" H 3050 6550 60  0000 C CNN
@@
 $EndComp
 $Comp
-L ULN2803A U7
+L ULN2803A U8
 U 1 1 565EE98E
 P 8000 2850
-F 0 "U7" H 7950 2350 50  0000 C CNN
+F 0 "U8" H 7950 2350 50  0000 C CNN
 F 1 "ULN2803A" H 8000 3400 50  0000 C CNN
 F 2 "" H 8000 2850 60  0000 C CNN
@@
 $EndComp
 $Comp
-L +5V #PWR65
+L +5V #PWR68
 U 1 1 5666DDAD
 P 9750 3450
-F 0 "#PWR65" H 9750 3540 20  0001 C CNN
+F 0 "#PWR68" H 9750 3540 20  0001 C CNN
 F 1 "+5V" H 9750 3540 30  0000 C CNN
 F 2 "" H 9750 3450 60  0000 C CNN
@@
 $EndComp
 $Comp
-L GND #PWR57
+L GND #PWR58
 U 1 1 5667DC7C
 P 5550 6250
-F 0 "#PWR57" H 5550 6000 50  0001 C CNN
+F 0 "#PWR58" H 5550 6000 50  0001 C CNN
 F 1 "GND" H 5550 6100 50  0000 C CNN
 F 2 "" H 5550 6250 50  0000 C CNN
@@
 $EndComp
 $Comp
-L +5V #PWR56
+L +5V #PWR57
 U 1 1 5667E681
 P 5450 2000
-F 0 "#PWR56" H 5450 1850 50  0001 C CNN
+F 0 "#PWR57" H 5450 1850 50  0001 C CNN
 F 1 "+5V" H 5450 2140 50  0000 C CNN
 F 2 "" H 5450 2000 50  0000 C CNN
@@
 NoConn ~ 5650 6150
 $Comp
-L GND #PWR59
+L GND #PWR62
 U 1 1 56680A85
 P 7250 3250
-F 0 "#PWR59" H 7250 3000 50  0001 C CNN
+F 0 "#PWR62" H 7250 3000 50  0001 C CNN
 F 1 "GND" H 7250 3100 50  0000 C CNN
 F 2 "" H 7250 3250 50  0000 C CNN
@@
 $EndComp
 $Comp
-L GND #PWR61
+L GND #PWR64
 U 1 1 56682AC8
 P 7900 1900
-F 0 "#PWR61" H 7900 1650 50  0001 C CNN
+F 0 "#PWR64" H 7900 1650 50  0001 C CNN
 F 1 "GND" H 7900 1750 50  0000 C CNN
 F 2 "" H 7900 1900 50  0000 C CNN
@@
 $EndComp
 $Comp
-L +5V #PWR66
+L +5V #PWR69
 U 1 1 566945A2
 P 11600 5350
-F 0 "#PWR66" H 11600 5200 50  0001 C CNN
+F 0 "#PWR69" H 11600 5200 50  0001 C CNN
 F 1 "+5V" H 11600 5490 50  0000 C CNN
 F 2 "" H 11600 5350 50  0000 C CNN
@@
 $EndComp
 $Comp
-L GND #PWR58
+L GND #PWR59
 U 1 1 5669531F
 P 6250 8100
-F 0 "#PWR58" H 6250 7850 50  0001 C CNN
+F 0 "#PWR59" H 6250 7850 50  0001 C CNN
 F 1 "GND" H 6250 7950 50  0000 C CNN
 F 2 "" H 6250 8100 50  0000 C CNN
@@
 $EndComp
 $Comp
-L JHD-162A U8
+L JHD-162A U9
 U 1 1 5666E893
 P 13100 6050
-F 0 "U8" H 11650 6650 60  0000 C CNN
+F 0 "U9" H 11650 6650 60  0000 C CNN
 F 1 "JHD-162A" H 14300 6650 60  0000 C CNN
 F 2 "" H 13100 6050 60  0000 C CNN
@@
 $EndComp
 $Comp
-L GND #PWR67
+L GND #PWR70
 U 1 1 5669686B
 P 12050 7900
-F 0 "#PWR67" H 12050 7650 50  0001 C CNN
+F 0 "#PWR70" H 12050 7650 50  0001 C CNN
 F 1 "GND" H 12050 7750 50  0000 C CNN
 F 2 "" H 12050 7900 50  0000 C CNN
@@
 	0    -1   -1   0
 $EndComp
-Text Notes 5250 8400 0    60   ~ 0
-Powered by VCC
 NoConn ~ 8750 2750
 NoConn ~ 7250 2750
 NoConn ~ 11350 4350
 $Comp
-L 4067 U6
+L 4067 U7
 U 1 1 565EE92F
 P 5650 7350
-F 0 "U6" H 5900 8200 60  0000 C CNN
+F 0 "U7" H 5900 8200 60  0000 C CNN
 F 1 "4067" H 5950 6450 60  0000 C CNN
 F 2 "" H 5650 7350 60  0000 C CNN
@@
 $EndComp
 $Comp
-L GND #PWR55
+L GND #PWR56
 U 1 1 568A98D8
 P 4950 8800
-F 0 "#PWR55" H 4950 8550 50  0001 C CNN
+F 0 "#PWR56" H 4950 8550 50  0001 C CNN
 F 1 "GND" H 4950 8650 50  0000 C CNN
 F 2 "" H 4950 8800 50  0000 C CNN
@@
 NoConn ~ 6600 4050
 $Comp
-L CONN_01X02 P14
+L CONN_01X02 P10
 U 1 1 5669A8F7
 P 8300 3750
-F 0 "P14" H 8300 3900 50  0000 C CNN
+F 0 "P10" H 8300 3900 50  0000 C CNN
 F 1 "CONN_01X02" V 8400 3750 50  0000 C CNN
 F 2 "UART" H 8250 3600 50  0000 C CNN
@@
 $EndComp
 $Comp
-L GND #PWR64
+L GND #PWR67
 U 1 1 566A8FFF
 P 8550 7850
-F 0 "#PWR64" H 8550 7600 50  0001 C CNN
+F 0 "#PWR67" H 8550 7600 50  0001 C CNN
 F 1 "GND" H 8550 7700 50  0000 C CNN
 F 2 "" H 8550 7850 50  0000 C CNN
@@
 $EndComp
 $Comp
-L GND #PWR63
+L GND #PWR66
 U 1 1 568B30CE
 P 8550 5000
-F 0 "#PWR63" H 8550 4750 50  0001 C CNN
+F 0 "#PWR66" H 8550 4750 50  0001 C CNN
 F 1 "GND" H 8550 4850 50  0000 C CNN
 F 2 "" H 8550 5000 50  0000 C CNN
@@
 $EndComp
 $Comp
-L GND #PWR60
+L GND #PWR63
 U 1 1 568E5271
 P 7750 4150
-F 0 "#PWR60" H 7750 3900 50  0001 C CNN
+F 0 "#PWR63" H 7750 3900 50  0001 C CNN
 F 1 "GND" H 7750 4000 50  0000 C CNN
 F 2 "" H 7750 4150 50  0000 C CNN
@@
 $EndComp
 $Comp
-L GND #PWR62
+L GND #PWR65
 U 1 1 568E530C
 P 8000 4150
-F 0 "#PWR62" H 8000 3900 50  0001 C CNN
+F 0 "#PWR65" H 8000 3900 50  0001 C CNN
 F 1 "GND" H 8000 4000 50  0000 C CNN
 F 2 "" H 8000 4150 50  0000 C CNN
@@
 	8000 3850 8000 3800
 Connection ~ 8000 3800
+$Comp
+L VCC #PWR60
+U 1 1 5671E26C
+P 6550 8000
+F 0 "#PWR60" H 6550 8100 30  0001 C CNN
+F 1 "VCC" H 6550 8100 30  0000 C CNN
+F 2 "" H 6550 8000 60  0000 C CNN
+F 3 "" H 6550 8000 60  0000 C CNN
+	1    6550 8000
+	1    0    0    -1
+$EndComp
+$Comp
+L C C12
+U 1 1 5671E272
+P 6550 8150
+F 0 "C12" H 6575 8250 50  0000 L CNN
+F 1 "C" H 6575 8050 50  0000 L CNN
+F 2 "0.1uF" H 6588 8000 50  0000 C CNN
+F 3 "" H 6550 8150 50  0000 C CNN
+	1    6550 8150
+	1    0    0    -1
+$EndComp
+$Comp
+L GND #PWR61
+U 1 1 5671E279
+P 6550 8300
+F 0 "#PWR61" H 6550 8050 50  0001 C CNN
+F 1 "GND" H 6550 8150 50  0000 C CNN
+F 2 "" H 6550 8300 50  0000 C CNN
+F 3 "" H 6550 8300 50  0000 C CNN
+	1    6550 8300
+	1    0    0    -1
+$EndComp
 $EndSCHEMATC
