File: in_progress/trainer/hex.sch (KiCad schematic (older format))
At the start: 49 parts, among them IC1 ATMEGA16-P, P10 CONN_01X02, P9 CONN_02X08, Q3 2N3904, Q4 2N3904, Q5 2N3904, Q6 2N3904, SW21 DEC/HEX, SW22 SW_PUSH, SW23 SW_PUSH, U7 4067, U8 ULN2803A, U9 JHD-162A

Commit message: .
Parts:
- added P12: CONN_01X07, symbol CONN_01X07
- added P13: CONN_02X03, symbol CONN_02X03
Connections:
- net at IC1.22 ((SCL)PC0), U9.4 (RS): now also P12.1 (P1)
- net at IC1.23 ((SDA)PC1), U9.5 (R/W): now also P12.2 (P2)
- net at IC1.24 ((TCK)PC2), U9.6 (E): now also P12.3 (P3)
- net at IC1.25 ((TMS)PC3), U9.11 (DB4): now also P12.4 (P4)
- net at IC1.26 ((TDO)PC4), U9.12 (DB5): now also P12.5 (P5)
- net at IC1.27 ((TDI)PC5), U9.13 (DB6): now also P12.6 (P6)
- net at IC1.28 ((TOSC1)PC6), U9.14 (DB7): now also P12.7 (P7)
Changed lines of the file:
@@
 	1    0    0    -1
+$EndComp
+$Comp
+L R R41
+U 1 1 568B24E5
+P 8200 4950
+F 0 "R41" V 8280 4950 50  0000 C CNN
+F 1 "R" V 8200 4950 50  0000 C CNN
+F 2 "560R" V 8130 4950 50  0000 C CNN
+F 3 "" H 8200 4950 50  0000 C CNN
+	1    8200 4950
+	0    1    1    0
+$EndComp
+$Comp
+L Led_Small D18
+U 1 1 568B300A
+P 8450 4950
+F 0 "D18" H 8400 5075 50  0000 L CNN
+F 1 "Led_Small" H 8150 4850 50  0000 L CNN
+F 2 "" V 8450 4950 50  0000 C CNN
+F 3 "" V 8450 4950 50  0000 C CNN
+	1    8450 4950
+	-1   0    0    1
+$EndComp
+$Comp
+L GND #PWR66
+U 1 1 568B30CE
+P 8550 5000
+F 0 "#PWR66" H 8550 4750 50  0001 C CNN
+F 1 "GND" H 8550 4850 50  0000 C CNN
+F 2 "" H 8550 5000 50  0000 C CNN
+F 3 "" H 8550 5000 50  0000 C CNN
+	1    8550 5000
+	1    0    0    -1
+$EndComp
+$Comp
+L C C9
+U 1 1 568DF9AB
+P 4200 2700
+F 0 "C9" H 4225 2800 50  0000 L CNN
+F 1 "C" H 4225 2600 50  0000 L CNN
+F 2 "0.1uF" H 4050 2600 50  0000 C CNN
+F 3 "" H 4200 2700 50  0000 C CNN
+	1    4200 2700
+	1    0    0    -1
+$EndComp
+$Comp
+L R R42
+U 1 1 568E36BE
+P 8500 5550
+F 0 "R42" V 8450 5750 50  0000 C CNN
+F 1 "R" V 8500 5550 50  0000 C CNN
+F 2 "1k8" V 8450 5350 50  0000 C CNN
+F 3 "" H 8500 5550 50  0000 C CNN
+	1    8500 5550
+	0    1    1    0
+$EndComp
+$Comp
+L R R43
+U 1 1 568E393C
+P 8500 5650
+F 0 "R43" V 8450 5850 50  0000 C CNN
+F 1 "R" V 8500 5650 50  0000 C CNN
+F 2 "1k8" V 8450 5450 50  0000 C CNN
+F 3 "" H 8500 5650 50  0000 C CNN
+	1    8500 5650
+	0    1    1    0
+$EndComp
+$Comp
+L R R44
+U 1 1 568E39D0
+P 8500 5750
+F 0 "R44" V 8450 5950 50  0000 C CNN
+F 1 "R" V 8500 5750 50  0000 C CNN
+F 2 "1k8" V 8450 5550 50  0000 C CNN
+F 3 "" H 8500 5750 50  0000 C CNN
+	1    8500 5750
+	0    1    1    0
+$EndComp
+$Comp
+L R R45
+U 1 1 568E3A67
+P 8500 5850
+F 0 "R45" V 8450 6050 50  0000 C CNN
+F 1 "R" V 8500 5850 50  0000 C CNN
+F 2 "1k8" V 8450 5650 50  0000 C CNN
+F 3 "" H 8500 5850 50  0000 C CNN
+	1    8500 5850
+	0    1    1    0
+$EndComp
+$Comp
+L R R39
+U 1 1 568E50BC
+P 7750 4000
+F 0 "R39" V 7830 4000 50  0000 C CNN
+F 1 "R" V 7750 4000 50  0000 C CNN
+F 2 "10k" V 7680 4000 50  0000 C CNN
+F 3 "" H 7750 4000 50  0000 C CNN
+	1    7750 4000
+	1    0    0    -1
+$EndComp
+$Comp
+L R R40
+U 1 1 568E51CB
+P 8000 4000
+F 0 "R40" V 8080 4000 50  0000 C CNN
+F 1 "R" V 8000 4000 50  0000 C CNN
+F 2 "10k" V 7930 4000 50  0000 C CNN
+F 3 "" H 8000 4000 50  0000 C CNN
+	1    8000 4000
+	1    0    0    -1
+$EndComp
+$Comp
+L GND #PWR63
+U 1 1 568E5271
+P 7750 4150
+F 0 "#PWR63" H 7750 3900 50  0001 C CNN
+F 1 "GND" H 7750 4000 50  0000 C CNN
+F 2 "" H 7750 4150 50  0000 C CNN
+F 3 "" H 7750 4150 50  0000 C CNN
+	1    7750 4150
+	1    0    0    -1
+$EndComp
+$Comp
+L GND #PWR65
+U 1 1 568E530C
+P 8000 4150
+F 0 "#PWR65" H 8000 3900 50  0001 C CNN
+F 1 "GND" H 8000 4000 50  0000 C CNN
+F 2 "" H 8000 4150 50  0000 C CNN
+F 3 "" H 8000 4150 50  0000 C CNN
+	1    8000 4150
+	1    0    0    -1
+$EndComp
+$Comp
+L VCC #PWR60
+U 1 1 5671E26C
+P 6550 8000
+F 0 "#PWR60" H 6550 8100 30  0001 C CNN
+F 1 "VCC" H 6550 8100 30  0000 C CNN
+F 2 "" H 6550 8000 60  0000 C CNN
+F 3 "" H 6550 8000 60  0000 C CNN
+	1    6550 8000
+	1    0    0    -1
+$EndComp
+$Comp
+L C C12
+U 1 1 5671E272
+P 6550 8150
+F 0 "C12" H 6575 8250 50  0000 L CNN
+F 1 "C" H 6575 8050 50  0000 L CNN
+F 2 "0.1uF" H 6588 8000 50  0000 C CNN
+F 3 "" H 6550 8150 50  0000 C CNN
+	1    6550 8150
+	1    0    0    -1
+$EndComp
+$Comp
+L GND #PWR61
+U 1 1 5671E279
+P 6550 8300
+F 0 "#PWR61" H 6550 8050 50  0001 C CNN
+F 1 "GND" H 6550 8150 50  0000 C CNN
+F 2 "" H 6550 8300 50  0000 C CNN
+F 3 "" H 6550 8300 50  0000 C CNN
+	1    6550 8300
+	1    0    0    -1
+$EndComp
+$Comp
+L CONN_01X07 P12
+U 1 1 566F4B22
+P 10650 7600
+F 0 "P12" H 10650 8000 50  0000 C CNN
+F 1 "CONN_01X07" V 10750 7600 50  0000 C CNN
+F 2 "" H 10650 7600 50  0000 C CNN
+F 3 "" H 10650 7600 50  0000 C CNN
+	1    10650 7600
+	0    1    1    0
 $EndComp
 Wire Wire Line
@@
 Wire Wire Line
 	7050 3750 6600 3750
-$Comp
-L R R41
-U 1 1 568B24E5
-P 8200 4950
-F 0 "R41" V 8280 4950 50  0000 C CNN
-F 1 "R" V 8200 4950 50  0000 C CNN
-F 2 "560R" V 8130 4950 50  0000 C CNN
-F 3 "" H 8200 4950 50  0000 C CNN
-	1    8200 4950
-	0    1    1    0
-$EndComp
-$Comp
-L Led_Small D18
-U 1 1 568B300A
-P 8450 4950
-F 0 "D18" H 8400 5075 50  0000 L CNN
-F 1 "Led_Small" H 8150 4850 50  0000 L CNN
-F 2 "" V 8450 4950 50  0000 C CNN
-F 3 "" V 8450 4950 50  0000 C CNN
-	1    8450 4950
-	-1   0    0    1
-$EndComp
-$Comp
-L GND #PWR66
-U 1 1 568B30CE
-P 8550 5000
-F 0 "#PWR66" H 8550 4750 50  0001 C CNN
-F 1 "GND" H 8550 4850 50  0000 C CNN
-F 2 "" H 8550 5000 50  0000 C CNN
-F 3 "" H 8550 5000 50  0000 C CNN
-	1    8550 5000
-	1    0    0    -1
-$EndComp
 Wire Wire Line
 	8550 4950 8550 5000
@@
 Wire Wire Line
 	7300 7800 7900 7800
-$Comp
-L C C9
-U 1 1 568DF9AB
-P 4200 2700
-F 0 "C9" H 4225 2800 50  0000 L CNN
-F 1 "C" H 4225 2600 50  0000 L CNN
-F 2 "0.1uF" H 4050 2600 50  0000 C CNN
-F 3 "" H 4200 2700 50  0000 C CNN
-	1    4200 2700
-	1    0    0    -1
-$EndComp
 Wire Wire Line
 	5550 6150 5550 6250
@@
 	4200 2050 5450 2050
 Connection ~ 5450 2050
-$Comp
-L R R42
-U 1 1 568E36BE
-P 8500 5550
-F 0 "R42" V 8450 5750 50  0000 C CNN
-F 1 "R" V 8500 5550 50  0000 C CNN
-F 2 "1k8" V 8450 5350 50  0000 C CNN
-F 3 "" H 8500 5550 50  0000 C CNN
-	1    8500 5550
-	0    1    1    0
-$EndComp
-$Comp
-L R R43
-U 1 1 568E393C
-P 8500 5650
-F 0 "R43" V 8450 5850 50  0000 C CNN
-F 1 "R" V 8500 5650 50  0000 C CNN
-F 2 "1k8" V 8450 5450 50  0000 C CNN
-F 3 "" H 8500 5650 50  0000 C CNN
-	1    8500 5650
-	0    1    1    0
-$EndComp
-$Comp
-L R R44
-U 1 1 568E39D0
-P 8500 5750
-F 0 "R44" V 8450 5950 50  0000 C CNN
-F 1 "R" V 8500 5750 50  0000 C CNN
-F 2 "1k8" V 8450 5550 50  0000 C CNN
-F 3 "" H 8500 5750 50  0000 C CNN
-	1    8500 5750
-	0    1    1    0
-$EndComp
-$Comp
-L R R45
-U 1 1 568E3A67
-P 8500 5850
-F 0 "R45" V 8450 6050 50  0000 C CNN
-F 1 "R" V 8500 5850 50  0000 C CNN
-F 2 "1k8" V 8450 5650 50  0000 C CNN
-F 3 "" H 8500 5850 50  0000 C CNN
-	1    8500 5850
-	0    1    1    0
-$EndComp
 Wire Wire Line
 	6600 5150 7200 5150
@@
 Wire Wire Line
 	7300 3800 8100 3800
-$Comp
-L R R39
-U 1 1 568E50BC
-P 7750 4000
-F 0 "R39" V 7830 4000 50  0000 C CNN
-F 1 "R" V 7750 4000 50  0000 C CNN
-F 2 "10k" V 7680 4000 50  0000 C CNN
-F 3 "" H 7750 4000 50  0000 C CNN
-	1    7750 4000
-	1    0    0    -1
-$EndComp
-$Comp
-L R R40
-U 1 1 568E51CB
-P 8000 4000
-F 0 "R40" V 8080 4000 50  0000 C CNN
-F 1 "R" V 8000 4000 50  0000 C CNN
-F 2 "10k" V 7930 4000 50  0000 C CNN
-F 3 "" H 8000 4000 50  0000 C CNN
-	1    8000 4000
-	1    0    0    -1
-$EndComp
-$Comp
-L GND #PWR63
-U 1 1 568E5271
-P 7750 4150
-F 0 "#PWR63" H 7750 3900 50  0001 C CNN
-F 1 "GND" H 7750 4000 50  0000 C CNN
-F 2 "" H 7750 4150 50  0000 C CNN
-F 3 "" H 7750 4150 50  0000 C CNN
-	1    7750 4150
-	1    0    0    -1
-$EndComp
-$Comp
-L GND #PWR65
-U 1 1 568E530C
-P 8000 4150
-F 0 "#PWR65" H 8000 3900 50  0001 C CNN
-F 1 "GND" H 8000 4000 50  0000 C CNN
-F 2 "" H 8000 4150 50  0000 C CNN
-F 3 "" H 8000 4150 50  0000 C CNN
-	1    8000 4150
-	1    0    0    -1
-$EndComp
 Wire Wire Line
 	7750 3850 7750 3700
@@
 	8000 3850 8000 3800
 Connection ~ 8000 3800
-$Comp
-L VCC #PWR60
-U 1 1 5671E26C
-P 6550 8000
-F 0 "#PWR60" H 6550 8100 30  0001 C CNN
-F 1 "VCC" H 6550 8100 30  0000 C CNN
-F 2 "" H 6550 8000 60  0000 C CNN
-F 3 "" H 6550 8000 60  0000 C CNN
-	1    6550 8000
-	1    0    0    -1
-$EndComp
-$Comp
-L C C12
-U 1 1 5671E272
-P 6550 8150
-F 0 "C12" H 6575 8250 50  0000 L CNN
-F 1 "C" H 6575 8050 50  0000 L CNN
-F 2 "0.1uF" H 6588 8000 50  0000 C CNN
-F 3 "" H 6550 8150 50  0000 C CNN
-	1    6550 8150
-	1    0    0    -1
-$EndComp
-$Comp
-L GND #PWR61
-U 1 1 5671E279
-P 6550 8300
-F 0 "#PWR61" H 6550 8050 50  0001 C CNN
-F 1 "GND" H 6550 8150 50  0000 C CNN
-F 2 "" H 6550 8300 50  0000 C CNN
-F 3 "" H 6550 8300 50  0000 C CNN
-	1    6550 8300
-	1    0    0    -1
-$EndComp
+Wire Wire Line
+	10950 7400 10950 7000
+Connection ~ 10950 7000
+Wire Wire Line
+	10850 7400 10850 6900
+Connection ~ 10850 6900
+Wire Wire Line
+	10750 7400 10750 6800
+Connection ~ 10750 6800
+Wire Wire Line
+	10650 7400 10650 6300
+Connection ~ 10650 6300
+Wire Wire Line
+	10550 7400 10550 6200
+Connection ~ 10550 6200
+Wire Wire Line
+	10450 6100 10450 7400
+Connection ~ 10450 6100
+Wire Wire Line
+	10350 7400 10350 6000
+Connection ~ 10350 6000
+$Comp
+L CONN_02X03 P13
+U 1 1 566F6147
+P 10650 8400
+F 0 "P13" H 10650 8600 50  0000 C CNN
+F 1 "CONN_02X03" H 10650 8200 50  0000 C CNN
+F 2 "" H 10650 7200 50  0000 C CNN
+F 3 "" H 10650 7200 50  0000 C CNN
+	1    10650 8400
+	1    0    0    -1
+$EndComp
