File: in_progress/trainer/inputs.sch (KiCad schematic (older format))
At the start: 45 parts

Commit message: .
Parts:
- gave numbers to parts that had none: 42
Connections:
- net at U6.1 (OEa), U6.19 (OEb): now also U5.2; no longer U5.10
- net at SW17.2: now also U5.1; no longer U5.11

Commit message: .
Parts:
- C3, C4, C5, C6, C7: footprint 10nF -> 1uF
- R22, R23, R24, R25, R26: footprint 10k -> 20k
Changed lines of the file:
@@
 F 0 "R23" V 7680 3800 50  0000 C CNN
 F 1 "R" V 7600 3800 50  0000 C CNN
-F 2 "10k" V 7650 3950 30  0000 C CNN
+F 2 "20k" V 7650 3950 30  0000 C CNN
 F 3 "" H 7600 3800 30  0000 C CNN
 	1    7600 3800
@@
 F 0 "C4" H 7625 4350 50  0000 L CNN
 F 1 "C" H 7625 4150 50  0000 L CNN
-F 2 "10nF" H 7500 4150 30  0000 C CNN
+F 2 "1uF" H 7500 4150 30  0000 C CNN
 F 3 "" H 7600 4250 60  0000 C CNN
 	1    7600 4250
@@
 F 0 "R24" V 7680 5050 50  0000 C CNN
 F 1 "R" V 7600 5050 50  0000 C CNN
-F 2 "10k" V 7700 5150 30  0000 C CNN
+F 2 "20k" V 7700 5150 30  0000 C CNN
 F 3 "" H 7600 5050 30  0000 C CNN
 	1    7600 5050
@@
 F 0 "C5" H 7625 5600 50  0000 L CNN
 F 1 "C" H 7625 5400 50  0000 L CNN
-F 2 "10nF" H 7500 5400 30  0000 C CNN
+F 2 "1uF" H 7500 5400 30  0000 C CNN
 F 3 "" H 7600 5500 60  0000 C CNN
 	1    7600 5500
@@
 F 0 "R25" V 10280 3800 50  0000 C CNN
 F 1 "R" V 10200 3800 50  0000 C CNN
-F 2 "10k" V 10250 3950 30  0000 C CNN
+F 2 "20k" V 10250 3950 30  0000 C CNN
 F 3 "" H 10200 3800 30  0000 C CNN
 	1    10200 3800
@@
 F 0 "C6" H 10225 4350 50  0000 L CNN
 F 1 "C" H 10225 4150 50  0000 L CNN
-F 2 "10nF" H 10100 4150 30  0000 C CNN
+F 2 "1uF" H 10100 4150 30  0000 C CNN
 F 3 "" H 10200 4250 60  0000 C CNN
 	1    10200 4250
@@
 F 0 "R26" V 10280 5050 50  0000 C CNN
 F 1 "R" V 10200 5050 50  0000 C CNN
-F 2 "10k" V 10150 5200 30  0000 C CNN
+F 2 "20k" V 10150 5200 30  0000 C CNN
 F 3 "" H 10200 5050 30  0000 C CNN
 	1    10200 5050
@@
 F 0 "C7" H 10225 5600 50  0000 L CNN
 F 1 "C" H 10225 5400 50  0000 L CNN
-F 2 "10nF" H 10100 5400 30  0000 C CNN
+F 2 "1uF" H 10100 5400 30  0000 C CNN
 F 3 "" H 10200 5500 60  0000 C CNN
 	1    10200 5500
@@
 F 0 "R22" V 5430 4900 50  0000 C CNN
 F 1 "R" V 5350 4900 50  0000 C CNN
-F 2 "10k" V 5400 5050 30  0000 C CNN
+F 2 "20k" V 5400 5050 30  0000 C CNN
 F 3 "" H 5350 4900 30  0000 C CNN
 	1    5350 4900
@@
 F 0 "C3" H 5375 5450 50  0000 L CNN
 F 1 "C" H 5375 5250 50  0000 L CNN
-F 2 "10nF" H 5250 5250 30  0000 C CNN
+F 2 "1uF" H 5250 5250 30  0000 C CNN
 F 3 "" H 5350 5350 60  0000 C CNN
 	1    5350 5350

Commit message: .
Parts:
- removed C3: C, 1uF, symbol C-RESCUE-trainer
- removed P9: CONN_01X08, Buffered switches, symbol CONN_01X08
- removed R22: R, 20k, symbol R-RESCUE-trainer
- removed SW17: SW_PUSH, symbol SW_PUSH
- removed unit 1 of U5
- removed U6: 74HC244, symbol 74LS244
- added P10: CONN_01X08, Unbuffered switches, symbol CONN_01X08
- C5: renamed from C4; footprint 1uF -> 10uF
- C6: renamed from C5; footprint 1uF -> 10uF
- C7: renamed from C6; footprint 1uF -> 10uF
- C8: renamed from C7; footprint 1uF -> 10uF
- R19: renamed from R23; footprint 20k -> 10k
- R20: renamed from R24; footprint 20k -> 10k
- R21: renamed from R25; footprint 20k -> 10k
- R22: renamed from R26; footprint 20k -> 10k
- renumbered P10 to P11, P11 to P12, P8 to P9, SW18 to SW17, SW19 to SW18, SW20 to SW19, SW21 to SW20, U7 to U4
Connections:
- net at SW18.2: now also U5.1; no longer U5.3
- net at SW19.2: now also U5.3; no longer U5.5
- net at SW20.2: now also U5.5; no longer U5.9
- net at P12.2: now also U5.4; no longer U5.6
- net at P12.3: now also U5.2; no longer U5.4
- net at P12.4: now also U5.6; no longer U5.8
- net at SW9.2: now also P10.1 (P1)
- net at SW10.2: now also P10.2 (P2)
- net at SW11.2: now also P10.3 (P3)
- net at SW12.2: now also P10.4 (P4)
- net at SW13.2: now also P10.5 (P5)
- net at SW14.2: now also P10.6 (P6)
- net at SW15.2: now also P10.7 (P7)
- net at SW16.2: now also P10.8 (P8)

Commit message: .
Parts:
- removed P10, P9: CONN_01X08, Unbuffered switches, symbol CONN_01X08
- added C11: C, 0.1uF, symbol C
- added P6: CONN_02X08, symbol CONN_02X08
- renumbered P11 to P7, P12 to P8, U4 to U5, U5 to U6
Connections:
- net GND: now also RV1.1, RV2.1, RV3.1, RV4.1, C11.2
- net GNDREF: no longer RV1.1, RV2.1, RV3.1, RV4.1
- net VCC: now also C11.1
- net at SW1.2: now also P6.1 (P1)
- net at SW2.2: now also P6.3 (P3)
- net at SW3.2: now also P6.5 (P5)
- net at SW4.2: now also P6.7 (P7)
- net at SW5.2: now also P6.9 (P9)
- net at SW6.2: now also P6.11 (P11)
- net at SW7.2: now also P6.13 (P13)
- net at SW8.2: now also P6.15 (P15)
- net at SW9.2: now also P6.2 (P2)
- net at SW10.2: now also P6.4 (P4)
- net at SW11.2: now also P6.6 (P6)
- net at SW12.2: now also P6.8 (P8)
- net at SW13.2: now also P6.10 (P10)
- net at SW14.2: now also P6.12 (P12)
- net at SW15.2: now also P6.14 (P14)
- net at SW16.2: now also P6.16 (P16)
Other:
- moved on the sheet: C5, C6, C7, C8, P7, P8, R19, R20, R21, R22, RV1, RV2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
