File: in_progress/trainer/trainer.sch (KiCad schematic (older format))
At the start: 58 parts

Commit message: .
Parts:
- gave numbers to parts that had none: 58

Commit message: .
Parts:
- removed P1: CONN_01X04, RELAYS, symbol CONN_01X04
- removed R1, R2, R3, R4: R, 220R, symbol R-RESCUE-trainer
- removed S2, S3, S4: RELAY_SPDT, symbol RELAY_SPDT
- removed U1: ULN2803A, symbol ULN2803A
- added D?: D, 1N4007, symbol D
- added P?: CONN_01X01, symbol CONN_01X01
- added Q?: 2N3904, TO92, symbol PN2222A-RESCUE-trainer
- added R?: R, 2k2, symbol R-RESCUE-trainer
Connections:
- net labels removed: R2_CLOSED, R2_COM, R2_OPEN, R3_CLOSED, R3_COM, R3_OPEN, R4_CLOSED, R4_COM, R4_OPEN
- wire segments 123 -> 109
Other:
- moved on the sheet: S1
Changed lines of the file:
@@
 F1 "inputs.sch" 60
 $EndSheet
-$Comp
-L RELAY_SPDT S1
-U 1 1 56568F0F
-P 4700 4450
-F 0 "S1" H 4700 4150 60  0000 C CNN
-F 1 "RELAY_SPDT" H 4700 4050 60  0000 C CNN
-F 2 "" H 4700 4450 60  0000 C CNN
-F 3 "" H 4700 4450 60  0000 C CNN
-	1    4700 4450
-	1    0    0    -1
-$EndComp
-$Comp
-L CONN_01X04 P1
-U 1 1 5656959C
-P 1250 4900
-F 0 "P1" H 1250 5150 50  0000 C CNN
-F 1 "CONN_01X04" V 1350 4900 50  0000 C CNN
-F 2 "RELAYS" H 1350 5250 60  0000 C CNN
-F 3 "" H 1250 4900 60  0000 C CNN
-	1    1250 4900
-	-1   0    0    1
-$EndComp
-Text GLabel 5150 4300 2    60   Input ~ 0
+Text GLabel 4250 5000 2    60   Input ~ 0
 R1_CLOSED
-Text GLabel 5150 4450 2    60   Input ~ 0
+Text GLabel 4250 5150 2    60   Input ~ 0
 R1_COM
-Text GLabel 5150 4600 2    60   Input ~ 0
+Text GLabel 4250 5300 2    60   Input ~ 0
 R1_OPEN
-$Comp
-L RELAY_SPDT S2
-U 1 1 5656BF1B
-P 4700 5250
-F 0 "S2" H 4700 4950 60  0000 C CNN
-F 1 "RELAY_SPDT" H 4700 4850 60  0000 C CNN
-F 2 "" H 4700 5250 60  0000 C CNN
-F 3 "" H 4700 5250 60  0000 C CNN
-	1    4700 5250
-	1    0    0    -1
-$EndComp
-Text GLabel 5150 5100 2    60   Input ~ 0
-R2_CLOSED
-Text GLabel 5150 5250 2    60   Input ~ 0
-R2_COM
-Text GLabel 5150 5400 2    60   Input ~ 0
-R2_OPEN
-$Comp
-L RELAY_SPDT S3
-U 1 1 5656C278
-P 4700 6050
-F 0 "S3" H 4700 5750 60  0000 C CNN
-F 1 "RELAY_SPDT" H 4700 5650 60  0000 C CNN
-F 2 "" H 4700 6050 60  0000 C CNN
-F 3 "" H 4700 6050 60  0000 C CNN
-	1    4700 6050
-	1    0    0    -1
-$EndComp
-Text GLabel 5150 5900 2    60   Input ~ 0
-R3_CLOSED
-Text GLabel 5150 6050 2    60   Input ~ 0
-R3_COM
-Text GLabel 5150 6200 2    60   Input ~ 0
-R3_OPEN
-$Comp
-L RELAY_SPDT S4
-U 1 1 5656C28D
-P 4700 6850
-F 0 "S4" H 4700 6550 60  0000 C CNN
-F 1 "RELAY_SPDT" H 4700 6450 60  0000 C CNN
-F 2 "" H 4700 6850 60  0000 C CNN
-F 3 "" H 4700 6850 60  0000 C CNN
-	1    4700 6850
-	1    0    0    -1
-$EndComp
-Text GLabel 5150 6700 2    60   Input ~ 0
-R4_CLOSED
-Text GLabel 5150 6850 2    60   Input ~ 0
-R4_COM
-Text GLabel 5150 7000 2    60   Input ~ 0
-R4_OPEN
 $Comp
 L LM7805 U2
@@
 $EndComp
 $Comp
-L R-RESCUE-trainer R1
-U 1 1 5659DCCE
-P 3200 4750
-F 0 "R1" V 3150 4900 50  0000 C CNN
-F 1 "R" V 3200 4750 50  0000 C CNN
-F 2 "220R" V 3150 4550 30  0000 C CNN
-F 3 "" H 3200 4750 30  0000 C CNN
-	1    3200 4750
-	0    1    1    0
-$EndComp
-$Comp
-L R-RESCUE-trainer R2
-U 1 1 5659E1A6
-P 3200 4850
-F 0 "R2" V 3150 5000 50  0000 C CNN
-F 1 "R" V 3200 4850 50  0000 C CNN
-F 2 "220R" V 3150 4650 30  0000 C CNN
-F 3 "" H 3200 4850 30  0000 C CNN
-	1    3200 4850
-	0    1    1    0
-$EndComp
-$Comp
-L R-RESCUE-trainer R3
-U 1 1 5659E1E3
-P 3200 4950
-F 0 "R3" V 3150 5100 50  0000 C CNN
-F 1 "R" V 3200 4950 50  0000 C CNN
-F 2 "220R" V 3150 4750 30  0000 C CNN
-F 3 "" H 3200 4950 30  0000 C CNN
-	1    3200 4950
-	0    1    1    0
-$EndComp
-$Comp
-L R-RESCUE-trainer R4
-U 1 1 5659E227
-P 3200 5050
-F 0 "R4" V 3150 5200 50  0000 C CNN
-F 1 "R" V 3200 5050 50  0000 C CNN
-F 2 "220R" V 3150 4850 30  0000 C CNN
-F 3 "" H 3200 5050 30  0000 C CNN
-	1    3200 5050
-	0    1    1    0
-$EndComp
-$Comp
-L ULN2803A U1
-U 1 1 5659B908
-P 2200 5150
-F 0 "U1" H 2150 4650 50  0000 C CNN
-F 1 "ULN2803A" H 2200 5700 50  0000 C CNN
-F 2 "" H 2200 5150 60  0000 C CNN
-F 3 "" H 2200 5150 60  0000 C CNN
-	1    2200 5150
-	1    0    0    -1
-$EndComp
-$Comp
 L +5V #PWR8
 U 1 1 565A0518
-P 3950 3900
-F 0 "#PWR8" H 3950 3750 50  0001 C CNN
-F 1 "+5V" H 3950 4040 50  0000 C CNN
-F 2 "" H 3950 3900 60  0000 C CNN
-F 3 "" H 3950 3900 60  0000 C CNN
-	1    3950 3900
-	1    0    0    -1
-$EndComp
-$Comp
-L GNDREF #PWR3
-U 1 1 565A1ACC
-P 1450 5650
-F 0 "#PWR3" H 1450 5400 50  0001 C CNN
-F 1 "GNDREF" H 1450 5500 50  0000 C CNN
-F 2 "" H 1450 5650 60  0000 C CNN
-F 3 "" H 1450 5650 60  0000 C CNN
-	1    1450 5650
-	1    0    0    -1
-$EndComp
-$Comp
-L +5V #PWR6
-U 1 1 565A1B8D
-P 3300 5400
-F 0 "#PWR6" H 3300 5250 50  0001 C CNN
-F 1 "+5V" H 3300 5540 50  0000 C CNN
-F 2 "" H 3300 5400 60  0000 C CNN
-F 3 "" H 3300 5400 60  0000 C CNN
-	1    3300 5400
+P 3250 4700
+F 0 "#PWR8" H 3250 4550 50  0001 C CNN
+F 1 "+5V" H 3250 4840 50  0000 C CNN
+F 2 "" H 3250 4700 60  0000 C CNN
+F 3 "" H 3250 4700 60  0000 C CNN
+	1    3250 4700
 	1    0    0    -1
 $EndComp
@@
 	3500 2850 3500 2500
 Wire Wire Line
-	3950 3900 3950 6550
-Wire Wire Line
-	3950 4150 4150 4150
-Wire Wire Line
-	3950 4950 4150 4950
-Connection ~ 3950 4150
-Wire Wire Line
-	3950 5750 4150 5750
-Connection ~ 3950 4950
-Wire Wire Line
-	3950 6550 4150 6550
-Connection ~ 3950 5750
-Wire Wire Line
-	4150 4750 3450 4750
-Wire Wire Line
-	4150 5550 3850 5550
-Wire Wire Line
-	3850 5550 3850 4850
-Wire Wire Line
-	3850 4850 3450 4850
-Wire Wire Line
-	4150 6350 3750 6350
-Wire Wire Line
-	3750 6350 3750 4950
-Wire Wire Line
-	3750 4950 3450 4950
-Wire Wire Line
-	4150 7150 3650 7150
-Wire Wire Line
-	3650 7150 3650 5050
-Wire Wire Line
-	3650 5050 3450 5050
-Wire Wire Line
-	1450 5650 1450 5550
-Wire Wire Line
-	2950 5550 3300 5550
-Wire Wire Line
-	3300 5550 3300 5400
-Wire Wire Line
 	1350 1000 1350 1200
 Wire Wire Line
@@
 Wire Notes Line
 	4900 3550 4900 600
+$Comp
+L PN2222A-RESCUE-trainer Q?
+U 1 1 568E687A
+P 3150 5900
+F 0 "Q?" H 3150 5752 40  0000 R CNN
+F 1 "2N3904" H 3150 6050 40  0000 R CNN
+F 2 "TO92" H 3050 6002 29  0000 C CNN
+F 3 "~" H 3150 5900 60  0000 C CNN
+	1    3150 5900
+	1    0    0    -1
+$EndComp
+$Comp
+L R-RESCUE-trainer R?
+U 1 1 568E6880
+P 2700 5900
+F 0 "R?" V 2650 6050 50  0000 C CNN
+F 1 "R" V 2700 5900 50  0000 C CNN
+F 2 "2k2" V 2650 5700 30  0000 C CNN
+F 3 "" H 2700 5900 30  0000 C CNN
+	1    2700 5900
+	0    1    1    0
+$EndComp
+$Comp
+L GND #PWR?
+U 1 1 568E6886
+P 3250 6100
+F 0 "#PWR?" H 3250 5850 50  0001 C CNN
+F 1 "GND" H 3250 5950 50  0000 C CNN
+F 2 "" H 3250 6100 50  0000 C CNN
+F 3 "" H 3250 6100 50  0000 C CNN
+	1    3250 6100
+	1    0    0    -1
+$EndComp
+$Comp
+L D D?
+U 1 1 568E6A1E
+P 3100 5150
+F 0 "D?" H 3100 5250 50  0000 C CNN
+F 1 "D" H 3100 5050 50  0000 C CNN
+F 2 "1N4007" H 3100 5150 50  0000 C CNN
+F 3 "" H 3100 5150 50  0000 C CNN
+	1    3100 5150
+	0    1    1    0
+$EndComp
+$Comp
+L RELAY_SPDT S1
+U 1 1 56568F0F
+P 3800 5150
+F 0 "S1" H 3800 4850 60  0000 C CNN
+F 1 "RELAY_SPDT" H 3800 4750 60  0000 C CNN
+F 2 "" H 3800 5150 60  0000 C CNN
+F 3 "" H 3800 5150 60  0000 C CNN
+	1    3800 5150
+	1    0    0    -1
+$EndComp
+Wire Wire Line
+	3250 5300 3250 5700
+Wire Wire Line
+	3250 4700 3250 5000
+Wire Wire Line
+	3250 5300 3100 5300
+Connection ~ 3250 5450
+Wire Wire Line
+	3250 5000 3100 5000
+Connection ~ 3250 4850
+$Comp
+L CONN_01X01 P?
+U 1 1 568E752E
+P 2250 5900
+F 0 "P?" H 2250 6000 50  0000 C CNN
+F 1 "CONN_01X01" V 2350 5900 50  0000 C CNN
+F 2 "" H 2250 5900 50  0000 C CNN
+F 3 "" H 2250 5900 50  0000 C CNN
+	1    2250 5900
+	-1   0    0    1
+$EndComp
 $EndSCHEMATC

Commit message: .
Parts:
- added P?: CONN_01X01, symbol CONN_01X01
Other:
- note added: "Power to circuit"
- moved on the sheet: P2
Changed lines of the file:
@@
 L CONN_01X02 P2
 U 1 1 565A8A8C
-P 1700 1250
-F 0 "P2" H 1700 1400 50  0000 C CNN
-F 1 "CONN_01X02" V 1800 1250 50  0000 C CNN
-F 2 "Power from circuit" H 1950 950 60  0000 C CNN
-F 3 "" H 1700 1250 60  0000 C CNN
-	1    1700 1250
+P 1300 1500
+F 0 "P2" H 1300 1650 50  0000 C CNN
+F 1 "CONN_01X02" V 1400 1500 50  0000 C CNN
+F 2 "Power from circuit" H 1550 1200 60  0000 C CNN
+F 3 "" H 1300 1500 60  0000 C CNN
+	1    1300 1500
 	1    0    0    -1
 $EndComp
@@
 L VCC #PWR1
 U 1 1 565A8B1D
-P 1350 1000
-F 0 "#PWR1" H 1350 850 50  0001 C CNN
-F 1 "VCC" H 1350 1150 50  0000 C CNN
-F 2 "" H 1350 1000 60  0000 C CNN
-F 3 "" H 1350 1000 60  0000 C CNN
-	1    1350 1000
+P 950 1250
+F 0 "#PWR1" H 950 1100 50  0001 C CNN
+F 1 "VCC" H 950 1400 50  0000 C CNN
+F 2 "" H 950 1250 60  0000 C CNN
+F 3 "" H 950 1250 60  0000 C CNN
+	1    950  1250
 	1    0    0    -1
 $EndComp
@@
 L GNDREF #PWR2
 U 1 1 565A8FBD
-P 1350 1500
-F 0 "#PWR2" H 1350 1250 50  0001 C CNN
-F 1 "GNDREF" H 1350 1350 50  0000 C CNN
-F 2 "" H 1350 1500 60  0000 C CNN
-F 3 "" H 1350 1500 60  0000 C CNN
-	1    1350 1500
+P 950 1750
+F 0 "#PWR2" H 950 1500 50  0001 C CNN
+F 1 "GNDREF" H 950 1600 50  0000 C CNN
+F 2 "" H 950 1750 60  0000 C CNN
+F 3 "" H 950 1750 60  0000 C CNN
+	1    950  1750
 	1    0    0    -1
 $EndComp
@@
 	1650 2400 2100 2400
 Wire Wire Line
-	2900 2500 2900 2400
-Wire Wire Line
 	2900 2400 3500 2400
-Wire Wire Line
-	2100 2400 2100 2500
 Wire Wire Line
 	3250 2400 3250 2250
@@
 	1650 2850 3500 2850
 Wire Wire Line
-	2900 2850 2900 2800
-Wire Wire Line
 	2500 2700 2500 2950
-Connection ~ 2900 2850
 Connection ~ 2500 2850
-Wire Wire Line
-	2100 2850 2100 2800
-Connection ~ 2100 2850
 Wire Wire Line
 	3500 1500 3100 1500
@@
 	3500 2850 3500 2500
 Wire Wire Line
-	1350 1000 1350 1200
-Wire Wire Line
-	1350 1200 1500 1200
-Wire Wire Line
-	1350 1500 1350 1300
-Wire Wire Line
-	1350 1300 1500 1300
+	950  1250 950  1450
+Wire Wire Line
+	950  1450 1100 1450
+Wire Wire Line
+	950  1750 950  1550
+Wire Wire Line
+	950  1550 1100 1550
 Wire Wire Line
 	5950 1850 6050 1850
@@
 	-1   0    0    1
 $EndComp
+Wire Wire Line
+	2100 2400 2100 2450
+Wire Wire Line
+	2900 2450 2900 2400
+$Comp
+L CONN_01X01 P?
+U 1 1 566E190D
+P 1900 950
+F 0 "P?" H 1900 1050 50  0000 C CNN
+F 1 "CONN_01X01" V 2000 950 50  0000 C CNN
+F 2 "" H 1900 950 50  0000 C CNN
+F 3 "" H 1900 950 50  0000 C CNN
+	1    1900 950
+	-1   0    0    1
+$EndComp
+$Comp
+L +5V #PWR?
+U 1 1 566E2984
+P 2200 850
+F 0 "#PWR?" H 2200 700 50  0001 C CNN
+F 1 "+5V" H 2200 990 50  0000 C CNN
+F 2 "" H 2200 850 50  0000 C CNN
+F 3 "" H 2200 850 50  0000 C CNN
+	1    2200 850
+	1    0    0    -1
+$EndComp
+Wire Wire Line
+	2100 950  2200 950
+Wire Wire Line
+	2200 950  2200 850
+Text Notes 1950 1150 0    60   ~ 0
+Power to circuit
 $EndSCHEMATC

Commit message: .
Parts:
- removed P5: CONN_01X02, 5V to circuit, symbol CONN_01X02
- removed P6: CONN_01X03, symbol CONN_01X03
- removed P? (x2): CONN_01X01, symbol CONN_01X01
- removed SP1: SPEAKER, symbol SPEAKER
- added C1, C2: C, 0.1uF, symbol C-RESCUE-trainer
- added P?: CONN_01X01, Power to circuit, symbol CONN_01X01
- added P?: CONN_01X02, symbol CONN_01X02
- C3: renamed from C1; footprint 0.33uF -> 0.1uF
- gave numbers to parts that had none: 3
- renumbered C2 to C4, D9 to D10, D10 to D11, D11 to D12, D12 to D13, D13 to D14, D14 to D15, D15 to D16, D16 to D17, D1 to D2, D2 to D3, D3 to D4, D4 to D5, D5 to D6, D6 to D7, D7 to D8, D8 to D9, P2 to P1, P3 to P4, P4 to P5, P7 to P8, Q1 to Q2, R13 to R10, R14 to R11, R15 to R12, R16 to R13, R17 to R14, R18 to R15, R19 to R16, R20 to R17, R21 to R18, R5 to R2, R6 to R3, R7 to R4, R8 to R5, R9 to R6, R10 to R7, R11 to R8, R12 to R9, U2 to U1, U3 to U2, U4 to U3
Connections:
- net +5V: now also P?.1 (P1)
- net GNDREF: now also C4.2
- net at C3.1, CON1.1, U1.VI: now also C1.1, C2.1
- net at R2.2: now also P?.1 (P1)
- net at R1.2: now also P?.2 (P2)
Other:
- note removed: "Power to circuit"
- moved on the sheet: C3, C4, CON1, D1, P1, Q1, Q2, R1, R2, S1, U1, X1

Commit message: .
Parts:
- removed P1: CONN_01X02, Power from circuit, symbol CONN_01X02
- removed P4: CONN_01X03, USB, symbol CONN_01X03
- removed P?: CONN_01X01, Power to circuit, symbol CONN_01X01
- added C10: C, 220uF, symbol C-RESCUE-trainer
- added P11: CONN_01X03, symbol CONN_01X03
- added P2: CONN_02X02, symbol CONN_02X02
- added P3: CONN_01X04, symbol CONN_01X04
- added U2: LM3940, symbol LM7805
- gave numbers to parts that had none: 1
- renumbered P8 to P4, U2 to U3, U3 to U4
Connections:
- net +5V: now also P2.1 (P1), U2.VI
- net GNDREF: now also C1.2, C2.2, C3.2, C10.2, P2.4 (P4), P3.1 (P1), U2.GND
- net VCC: now also P2.2 (P2)
- net at P5.1 (VCC): now also P3.4 (P4)
- net at P5.2 (D-): now also P3.3 (P3)
- net at P5.3 (D+): now also P3.2 (P2)
- net at C1.1, C2.1, C3.1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: now also C10.1
- net R1_CLOSED: no longer names the net of S1.4 (NC)
- net R1_CLOSED: now also P11.1 (P1)
- net R1_COM: no longer names the net of S1.3
- net R1_COM: now also P11.2 (P2)
- net R1_OPEN: no longer names the net of S1.5 (NO)
- net R1_OPEN: now also P11.3 (P3)
- new net: P2.3 (P3), U2.VO
- no-connect marks 1 -> 3
Other:
- moved on the sheet: C1, C2, C3, C4, CON1, P5, U1

Commit message: .
Parts:
- added F1: FUSE, 1A, symbol FUSE
Connections:
- net at C1.1, C10.1, C2.1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: now also F1.2; no longer CON1.1
- new net: CON1.1, F1.1
Other:
- moved on the sheet: C1, C10, C2, C3, C4, CON1, P2, U1, U2
Changed lines of the file:
@@
 L C-RESCUE-trainer C3
 U 1 1 5657DDA5
-P 2900 2050
-F 0 "C3" H 2925 2150 50  0000 L CNN
-F 1 "C" H 2925 1950 50  0000 L CNN
-F 2 "0.1uF" H 2800 1950 30  0000 C CNN
-F 3 "" H 2900 2050 60  0000 C CNN
-	1    2900 2050
+P 3700 2150
+F 0 "C3" H 3725 2250 50  0000 L CNN
+F 1 "C" H 3725 2050 50  0000 L CNN
+F 2 "0.1uF" H 3600 2050 30  0000 C CNN
+F 3 "" H 3700 2150 60  0000 C CNN
+	1    3700 2150
 	1    0    0    -1
 $EndComp
@@
 L C-RESCUE-trainer C4
 U 1 1 5657DE9C
-P 3700 2050
-F 0 "C4" H 3725 2150 50  0000 L CNN
-F 1 "C" H 3725 1950 50  0000 L CNN
-F 2 "0.1uF" H 3850 1950 30  0000 C CNN
-F 3 "" H 3700 2050 60  0000 C CNN
-	1    3700 2050
+P 4500 2150
+F 0 "C4" H 4525 2250 50  0000 L CNN
+F 1 "C" H 4525 2050 50  0000 L CNN
+F 2 "0.1uF" H 4650 2050 30  0000 C CNN
+F 3 "" H 4500 2150 60  0000 C CNN
+	1    4500 2150
 	1    0    0    -1
 $EndComp
@@
 L GNDREF #PWR5
 U 1 1 5657E02B
-P 3300 2350
-F 0 "#PWR5" H 3300 2100 50  0001 C CNN
-F 1 "GNDREF" H 3300 2200 50  0000 C CNN
-F 2 "" H 3300 2350 60  0000 C CNN
-F 3 "" H 3300 2350 60  0000 C CNN
-	1    3300 2350
+P 4100 2450
+F 0 "#PWR5" H 4100 2200 50  0001 C CNN
+F 1 "GNDREF" H 4100 2300 50  0000 C CNN
+F 2 "" H 4100 2450 60  0000 C CNN
+F 3 "" H 4100 2450 60  0000 C CNN
+	1    4100 2450
 	1    0    0    -1
 $EndComp
@@
 L +5V #PWR6
 U 1 1 5657E06F
-P 3700 1150
-F 0 "#PWR6" H 3700 1000 50  0001 C CNN
-F 1 "+5V" H 3700 1290 50  0000 C CNN
-F 2 "" H 3700 1150 60  0000 C CNN
-F 3 "" H 3700 1150 60  0000 C CNN
-	1    3700 1150
+P 4500 1250
+F 0 "#PWR6" H 4500 1100 50  0001 C CNN
+F 1 "+5V" H 4500 1390 50  0000 C CNN
+F 2 "" H 4500 1250 60  0000 C CNN
+F 3 "" H 4500 1250 60  0000 C CNN
+	1    4500 1250
 	1    0    0    -1
 $EndComp
@@
 L BARREL_JACK CON1
 U 1 1 56587C69
-P 1400 1900
-F 0 "CON1" H 1400 2150 60  0000 C CNN
-F 1 "BARREL_JACK" H 1400 1700 60  0000 C CNN
-F 2 "7..12V" H 1400 1600 60  0000 C CNN
-F 3 "" H 1400 1900 60  0000 C CNN
-	1    1400 1900
+P 1700 2000
+F 0 "CON1" H 1700 2250 60  0000 C CNN
+F 1 "BARREL_JACK" H 1700 1800 60  0000 C CNN
+F 2 "7..12V" H 1700 1700 60  0000 C CNN
+F 3 "" H 1700 2000 60  0000 C CNN
+	1    1700 2000
 	1    0    0    -1
 $EndComp
@@
 L VCC #PWR8
 U 1 1 565A8B1D
-P 5250 1100
-F 0 "#PWR8" H 5250 950 50  0001 C CNN
-F 1 "VCC" H 5250 1250 50  0000 C CNN
-F 2 "" H 5250 1100 60  0000 C CNN
-F 3 "" H 5250 1100 60  0000 C CNN
-	1    5250 1100
+P 6050 1200
+F 0 "#PWR8" H 6050 1050 50  0001 C CNN
+F 1 "VCC" H 6050 1350 50  0000 C CNN
+F 2 "" H 6050 1200 60  0000 C CNN
+F 3 "" H 6050 1200 60  0000 C CNN
+	1    6050 1200
 	1    0    0    -1
 $EndComp
@@
 L GNDREF #PWR7
 U 1 1 565A8FBD
-P 5200 1550
-F 0 "#PWR7" H 5200 1300 50  0001 C CNN
-F 1 "GNDREF" H 5200 1400 50  0000 C CNN
-F 2 "" H 5200 1550 60  0000 C CNN
-F 3 "" H 5200 1550 60  0000 C CNN
-	1    5200 1550
-	1    0    0    -1
-$EndComp
-Text Notes 2300 2800 0    60   ~ 0
+P 6000 1650
+F 0 "#PWR7" H 6000 1400 50  0001 C CNN
+F 1 "GNDREF" H 6000 1500 50  0000 C CNN
+F 2 "" H 6000 1650 60  0000 C CNN
+F 3 "" H 6000 1650 60  0000 C CNN
+	1    6000 1650
+	1    0    0    -1
+$EndComp
+Text Notes 3100 2900 0    60   ~ 0
 Isolated power supply\n(powers internal LEDs, ICs)
 $Sheet
@@
 L C-RESCUE-trainer C2
 U 1 1 568F03CD
-P 2600 2050
-F 0 "C2" H 2625 2150 50  0000 L CNN
-F 1 "C" H 2625 1950 50  0000 L CNN
-F 2 "0.1uF" H 2500 1950 30  0000 C CNN
-F 3 "" H 2600 2050 60  0000 C CNN
-	1    2600 2050
+P 3400 2150
+F 0 "C2" H 3425 2250 50  0000 L CNN
+F 1 "C" H 3425 2050 50  0000 L CNN
+F 2 "0.1uF" H 3300 2050 30  0000 C CNN
+F 3 "" H 3400 2150 60  0000 C CNN
+	1    3400 2150
 	1    0    0    -1
 $EndComp
@@
 L C-RESCUE-trainer C1
 U 1 1 568F048E
-P 2300 2050
-F 0 "C1" H 2325 2150 50  0000 L CNN
-F 1 "C" H 2325 1950 50  0000 L CNN
-F 2 "0.1uF" H 2200 1950 30  0000 C CNN
-F 3 "" H 2300 2050 60  0000 C CNN
-	1    2300 2050
+P 3100 2150
+F 0 "C1" H 3125 2250 50  0000 L CNN
+F 1 "C" H 3125 2050 50  0000 L CNN
+F 2 "0.1uF" H 3000 2050 30  0000 C CNN
+F 3 "" H 3100 2150 60  0000 C CNN
+	1    3100 2150
 	1    0    0    -1
 $EndComp
@@
 L LM7805 U1
 U 1 1 5657C7C3
-P 3300 1850
-F 0 "U1" H 3450 1654 60  0000 C CNN
-F 1 "LM7805" H 3300 2050 60  0000 C CNN
-F 2 "" H 3300 1850 60  0000 C CNN
-F 3 "" H 3300 1850 60  0000 C CNN
-	1    3300 1850
+P 4100 1950
+F 0 "U1" H 4250 1754 60  0000 C CNN
+F 1 "LM7805" H 4100 2150 60  0000 C CNN
+F 2 "" H 4100 1950 60  0000 C CNN
+F 3 "" H 4100 1950 60  0000 C CNN
+	1    4100 1950
 	1    0    0    -1
 $EndComp
@@
 	7900 2150 7900 1500
 Wire Wire Line
-	1700 1800 2900 1800
-Wire Wire Line
-	3700 1150 3700 1850
-Wire Wire Line
-	1700 1900 1700 2250
-Connection ~ 1700 2000
-Wire Wire Line
-	3300 2100 3300 2350
-Connection ~ 3300 2250
+	2500 1900 3700 1900
+Wire Wire Line
+	4500 1250 4500 1950
+Wire Wire Line
+	4100 2200 4100 2450
+Connection ~ 4100 2350
 Wire Wire Line
 	7700 1800 7300 1800
@@
 Wire Wire Line
 	7600 1700 7600 1500
-Connection ~ 3700 1800
+Connection ~ 4500 1900
 Wire Wire Line
 	1550 6900 2050 6900
@@
 Connection ~ 2800 4000
 Wire Wire Line
-	2300 1850 2300 1800
-Connection ~ 2300 1800
-Wire Wire Line
-	2600 1850 2600 1800
-Connection ~ 2600 1800
-Wire Wire Line
-	2900 1800 2900 1850
+	3100 1950 3100 1900
+Connection ~ 3100 1900
+Wire Wire Line
+	3400 1950 3400 1900
+Connection ~ 3400 1900
+Wire Wire Line
+	3700 1900 3700 1950
 $Comp
 L CONN_01X02 P1
@@
 L CONN_02X02 P2
 U 1 1 566EE3C5
-P 4750 1350
-F 0 "P2" H 4750 1500 50  0000 C CNN
-F 1 "CONN_02X02" H 4750 1200 50  0000 C CNN
-F 2 "" H 4750 150 50  0000 C CNN
-F 3 "" H 4750 150 50  0000 C CNN
-	1    4750 1350
+P 5550 1450
+F 0 "P2" H 5550 1600 50  0000 C CNN
+F 1 "CONN_02X02" H 5550 1300 50  0000 C CNN
+F 2 "" H 5550 250 50  0000 C CNN
+F 3 "" H 5550 250 50  0000 C CNN
+	1    5550 1450
 	1    0    0    -1
 $EndComp
@@
 L LM7805 U2
 U 1 1 566EF639
-P 4100 1850
-F 0 "U2" H 4250 1654 50  0000 C CNN
-F 1 "LM3940" H 4100 2050 50  0000 C CNN
-F 2 "" H 4100 1850 50  0000 C CNN
-F 3 "" H 4100 1850 50  0000 C CNN
-	1    4100 1850
-	1    0    0    -1
-$EndComp
-Wire Wire Line
-	4500 1400 4500 1800
-Wire Wire Line
-	4500 1300 3700 1300
-Connection ~ 3700 1300
-Wire Wire Line
-	5000 1300 5250 1300
-Wire Wire Line
-	5250 1300 5250 1100
-Wire Wire Line
-	5000 1400 5200 1400
-Wire Wire Line
-	5200 1400 5200 1550
-Wire Wire Line
-	4100 2250 4100 2100
-Connection ~ 3700 2250
+P 4900 1950
+F 0 "U2" H 5050 1754 50  0000 C CNN
+F 1 "LM3940" H 4900 2150 50  0000 C CNN
+F 2 "" H 4900 1950 50  0000 C CNN
+F 3 "" H 4900 1950 50  0000 C CNN
+	1    4900 1950
+	1    0    0    -1
+$EndComp
+Wire Wire Line
+	5300 1500 5300 1900
+Wire Wire Line
+	5300 1400 4500 1400
+Connection ~ 4500 1400
+Wire Wire Line
+	5800 1400 6050 1400
+Wire Wire Line
+	6050 1400 6050 1200
+Wire Wire Line
+	5800 1500 6000 1500
+Wire Wire Line
+	6000 1500 6000 1650
+Wire Wire Line
+	4900 2350 4900 2200
+Connection ~ 4500 2350
 NoConn ~ 8950 4450
 NoConn ~ 8950 5700
-Connection ~ 2300 2250
-Connection ~ 2600 2250
-Connection ~ 2900 2250
+Connection ~ 3100 2350
+Connection ~ 3400 2350
+Connection ~ 3700 2350
 $Comp
 L CONN_01X04 P3
@@
 L C-RESCUE-trainer C10
 U 1 1 5671B0F2
-P 1950 2050
-F 0 "C10" H 1975 2150 50  0000 L CNN
-F 1 "C" H 1975 1950 50  0000 L CNN
-F 2 "220uF" H 1850 1950 30  0000 C CNN
-F 3 "" H 1950 2050 60  0000 C CNN
-	1    1950 2050
-	1    0    0    -1
-$EndComp
-Wire Wire Line
-	1700 2250 4100 2250
-Connection ~ 1950 2250
-Wire Wire Line
-	1950 1850 1950 1800
-Connection ~ 1950 1800
+P 2750 2150
+F 0 "C10" H 2775 2250 50  0000 L CNN
+F 1 "C" H 2775 2050 50  0000 L CNN
+F 2 "220uF" H 2650 2050 30  0000 C CNN
+F 3 "" H 2750 2150 60  0000 C CNN
+	1    2750 2150
+	1    0    0    -1
+$EndComp
+Wire Wire Line
+	2500 2350 4900 2350
+Connection ~ 2750 2350
+Wire Wire Line
+	2750 1950 2750 1900
+Connection ~ 2750 1900
+$Comp
+L FUSE F1
+U 1 1 566F2822
+P 2250 1900
+F 0 "F1" H 2350 1950 50  0000 C CNN
+F 1 "FUSE" H 2150 1850 50  0000 C CNN
+F 2 "1A" H 2250 2050 50  0000 C CNN
+F 3 "" H 2250 1900 50  0000 C CNN
+	1    2250 1900
+	1    0    0    -1
+$EndComp
+Wire Wire Line
+	2000 2000 2000 2100
+Wire Wire Line
+	2000 2100 2500 2100
+Wire Wire Line
+	2500 2100 2500 2350
 $EndSCHEMATC

Commit message: .
Parts:
- added C13: C, 47uF, symbol C-RESCUE-trainer
- added C14: C, 1uF, symbol C-RESCUE-trainer
Connections:
- net GNDREF: now also C13.2, C14.2
- net at P2.3 (P3), U2.VO: now also C13.1, C14.1
Other:
- note added: "3.3V"
- moved on the sheet: C1, C10, C2, C3, C4, CON1, F1, P2, U1, U2
